File: hardware/schematic/v1.0/CORE/CORE.kicad_sch (KiCad schematic)
At the start: 0 parts

Commit message: sch update commit
Parts:
- added BOOT_CFG1: CSW-2P, Counter:CSW DIP-2P, symbol Counter:CSW-2P
- added D1, D2: AZ1143-04F.R7G, Counter:DFN2510P10E, symbol Counter:AZ1045-04F.R7G
- added GE_PS1: HR911131A, Counter:HR911131A, symbol Counter:HR911131A_C
- added JTAG1: JTAG, Counter:DC3_14P_2_7_DIP, symbol Counter:Header 7X2
- added M1: ZYNQ7010&7020, Counter:ZYNQ7010&7020_CB, symbol Counter:ZYNQ7010&7020
- added R1, R2, R3, R4: 33R, Resistor_SMD:R_0402_1005Metric, symbol Device:R
- added U1: TXS02612RTWR, Counter:QFN24_RTW, symbol Counter:TXS02612RTWR
Connections:
- new net: JTAG1.10, R4.1
- new net: JTAG1.4, R1.1
- new net: JTAG1.6, R2.1
- new net: JTAG1.8, R3.1
- new net GND: JTAG1.1, JTAG1.11, JTAG1.13, JTAG1.3, JTAG1.5, JTAG1.7, JTAG1.9
- no-connect marks 0 -> 2
Other:
- note added: "MIO 4"
- note added: "MIO 5"

Commit message: sch update commit
Parts:
- added U2: SP3232, Counter:SOP16M, symbol Counter:MAX3232
Changed lines of the file:
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@@
+	)
+	(symbol
+		(lib_id "Counter:MAX3232")
+		(at 163.83 78.74 0)
+		(unit 1)
+		(body_style 1)
+		(exclude_from_sim no)
+		(in_bom yes)
+		(on_board yes)
+		(in_pos_files yes)
+		(dnp no)
+		(fields_autoplaced yes)
+		(property "Reference" "U2"
+			(at 176.53 71.12 0)
+			(show_name no)
+			(do_not_autoplace no)
+			(effects
+				(font
+					(size 1.8288 1.8288)
+				)
+			)
+		)
+		(property "Value" "SP3232"
+			(at 176.53 74.93 0)
+			(show_name no)
+			(do_not_autoplace no)
+			(effects
+				(font
+					(size 1.8288 1.8288)
+				)
+			)
+		)
+		(property "Footprint" "Counter:SOP16M"
+			(at 163.83 78.74 0)
+			(hide yes)
+			(show_name no)
+			(do_not_autoplace no)
+			(effects
+				(font
+					(size 1.27 1.27)
+				)
+			)
+		)
+		(property "Datasheet" ""
+			(at 163.83 78.74 0)
+			(hide yes)
+			(show_name no)
+			(do_not_autoplace no)
+			(effects
+				(font
+					(size 1.27 1.27)
+				)
+			)
+		)
+		(property "Description" ""
+			(at 163.83 78.74 0)
+			(hide yes)
+			(show_name no)
+			(do_not_autoplace no)
+			(effects
+				(font
+					(size 1.27 1.27)
+				)
+			)
+		)
+		(pin "5"
+		)
+		(pin "16"
+		)
+		(pin "4"
+		)
+		(pin "11"
+		)
+		(pin "13"
+		)
+		(pin "3"
+		)
+		(pin "7"
+		)
+		(pin "10"
+		)
+		(pin "1"
+		)
+		(pin "8"
+		)
+		(pin "15"
+		)
+		(pin "14"
+		)
+		(pin "6"
+		)
+		(pin "9"
+		)
+		(pin "2"
+		)
+		(pin "12"
+		)
+		(instances
+			(project "CORE"
+				(path "/c7438a17-8217-4925-98df-f8ca6801320f"
+					(reference "U2")
+					(unit 1)
+				)
+			)
+		)
 	)
 	(symbol

Commit message: sch update commit
Parts:
- added D3, D4, D5, D6: LED, symbol Device:LED
- added R10, R5, R6, R7, R8, R9: 499R, Resistor_SMD:R_0402_1005Metric, symbol Device:R
Connections:
- net GND: now also D3.1 (K), D4.1 (K), D5.1 (K), D6.1 (K)
- new net: D6.2 (A), R8.2
- new net: D4.2 (A), R6.2
- new net: D5.2 (A), R7.2
- new net: D3.2 (A), R5.2

Commit message: sch update commit
Parts:
- added R11, R12: 20K, Resistor_SMD:R_0402_1005Metric, symbol Device:R
- added R13, R14: 10K, Resistor_SMD:R_0402_1005Metric, symbol Device:R
- added U3: SD_Card, symbol Counter:SD_Card
- renumbered BOOT_CFG1 to BOOT_CFG
Connections:
- net GND: now also BOOT_CFG.1, BOOT_CFG.2
- net +3.3V: now reaches JTAG1.2
- net +3.3V: now also R13.2, R14.2
- net PS_LED1: now reaches R8.1
- net FPGA_TDI: now reaches R4.2
- net PL_LED1: now reaches R6.1
- net FPGA_TDO: now reaches R3.2
- net FPGA_TCK: now reaches R2.2
- net PL_LED0: now reaches R5.1
- net at BOOT_CFG.3: now also R12.1, R14.1
- net at BOOT_CFG.4: now also R11.1, R13.1
- net PS_LED0: now reaches R7.1
- net FPGA_TMS: now reaches R1.2
- new net BOOT_MODE0: R11.2
- new net BOOT_MODE1: R12.2
Other:
- moved on the sheet: BOOT_CFG

Commit message: sch update commit
Parts:
- added C1, C2, C3: 100nF, Capacitor_SMD:C_0402_1005Metric, symbol Device:C
- added R15: 4.7K, Resistor_SMD:R_0402_1005Metric, symbol Device:R
Connections:
- net +3.3V: now also R10.2, R9.1, U1.17 (VCCB1), U1.21 (VCCB0), C2.2
- net GND: now also D1.3 (GND), D1.8 (GND), D2.3 (GND), D2.8 (GND), GE_PS1.15 (GND), GE_PS1.16 (GND), U1.11 (GND2), U1.2 (GND1), U1.25 (EPAD), C1.2, C2.1, C3.1, R15.2
- net +5V: now reaches M1.J1_1 (1)
- net +5V: now also M1.J1_2 (2), M1.J1_3 (3), M1.J1_4 (4), M1.J1_5 (5), M1.J1_6 (6), M1.J1_7 (7), M1.J1_8 (8)
- net at R9.2: now also GE_PS1.14 (YA)
- net SD_D2: now reaches U1.1 (DAT2A)
- net at U1.24 (SEL): now also R15.1
- net SD_D3: now reaches U1.3 (DAT3A)
- net SD_CMD: now reaches U1.4 (CMDA)
- net +1.8V: now reaches U1.5 (VCCA)
- net +1.8V: now also C3.2
- net SD_D0: now reaches U1.6 (DAT0A)
- net SD_D1: now reaches U1.7 (DAT1A)
- net SD_CLK: now reaches U1.9 (CLKA)
- net at R10.1: now also GE_PS1.11 (GA)
- net at D2.10 (NC): now also GE_PS1.7 (TX3+)
- net at D2.6 (NC): now also GE_PS1.10 (TX4-)
- net at D2.7 (NC): now also GE_PS1.9 (TX4+)
- net at D2.9 (NC): now also GE_PS1.8 (TX3-)
- net at GE_PS1.1 (TX1+): now also D1.10 (NC)
- net at GE_PS1.2 (TX1-): now also D1.9 (NC)
- net at GE_PS1.3 (TX2+): now also D1.7 (NC)
- net at GE_PS1.4 (TX2-): now also D1.6 (NC)
- net at GE_PS1.5 (CT1): now also GE_PS1.6 (CT2), C1.1
- no-connect marks 2 -> 8
Other:
- moved on the sheet: D1, D2, R10, R9

Commit message: sch update commit
Parts:
- added R16: 330, Resistor_SMD:R_0402_1005Metric, symbol Device:R
- added R17: 0, Resistor_SMD:R_0402_1005Metric, symbol Device:R
- added R18: 10K, Resistor_SMD:R_0402_1005Metric, symbol Device:R
Connections:
- net +3.3V: now also R18.1
- net GND: now also U3.10 (GND), U3.11 (GND), U3.12 (GND), U3.13 (GND), U3.6 (VSS)
- net PL_LED0: now also M1.J2_44 (44)
- net PL_LED1: now also M1.J2_55 (55)
- net PS_LED0: now also M1.J2_92 (92)
- net PS_LED1: now also M1.J2_95 (95)
- net at U1.19 (CLKB0): now also U3.5 (CLK/SLCK)
- net at U3.9 (CD/SW): now also R16.2
- new net: R16.1, R17.2, R18.2
- new net SD_CD: R17.1
Other:
- moved on the sheet: C2, C3, D3, D4, D5, D6, R15, R5, R6, R7, R8, U1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

Commit message: sch update commit
Parts:
- added C4, C5: 10uF, Capacitor_SMD:C_0402_1005Metric, symbol Device:C
- added R19, R20, R21, R22, R23: 4.7K, Resistor_SMD:R_0402_1005Metric, symbol Device:R
Connections:
- net +3.3V: now also U3.4 (VDD), C4.1, C5.1, R19.1, R20.1, R21.1, R22.1, R23.1
- net BOOT_MODE0: now also M1.J2_81 (81)
- net BOOT_MODE1: now also M1.J2_79 (79)
- net FPGA_TCK: now also M1.J2_99 (99)
- net FPGA_TDI: now also M1.J2_98 (98)
- net FPGA_TDO: now also M1.J2_97 (97)
- net FPGA_TMS: now also M1.J2_100 (100)
- net GND: now also C4.2, C5.2
- net SD_CD: now also M1.J2_91 (91)
- net SD_CLK: now also M1.J2_80 (80)
- net SD_CMD: now also M1.J2_78 (78)
- net SD_D0: now also M1.J2_82 (82)
- net SD_D1: now also M1.J2_84 (84)
- net SD_D2: now also M1.J2_86 (86)
- net SD_D3: now also M1.J2_88 (88)
- net at U1.16 (DAT1B0): now also U3.8 (DAT1), R19.2
- net at U1.18 (DAT0B0): now also U3.7 (DAT0/SDO), R20.2
- net at U1.20 (CMDB0): now also U3.3 (CMD/SDI), R21.2
- net at U1.22 (DAT3B0): now also U3.2 (CD/DAT3/CS), R22.2
- net at U1.23 (DAT2B0): now also U3.1 (DAT2), R23.2
Other:
- moved on the sheet: C2

Commit message: sch update commit
Parts:
- added C10, C6, C7, C8, C9: 100nF, Capacitor_SMD:C_0402_1005Metric, symbol Device:C
- added J1: Conn_01x03_Socket, Connector_PinHeader_2.54mm:PinHeader_1x03_P2.54mm_Vertical, symbol Connector:Conn_01x03_Socket
Connections:
- net +3.3V: now also U2.16 (VCC), C6.2, C7.2
- net GND: now also U2.15 (GND), C10.2, C7.1, J1.1 (Pin_1)
- net PS_I2C_SDA: now reaches M1.J2_65 (65)
- net PS_I2C_SDA: now also M1.J2_70 (70)
- net PS_UART1_TXD: now reaches M1.J2_87 (87)
- net PS_UART1_TXD: now also U2.10 (DIN2)
- net PS_UART1_RXD: now reaches M1.J2_89 (89)
- net PS_UART1_RXD: now also U2.9 (ROUT2)
- net at U2.1 (C1+): now also C8.2
- net at U2.2 (V+): now also C6.1
- net at U2.3 (C1-): now also C8.1
- net at U2.4 (C2+): now also C9.2
- net at U2.5 (C2-): now also C9.1
- net at U2.6 (V-): now also C10.1
- net at U2.7 (DOUT2): now also J1.2 (Pin_2)
- net at U2.8 (RIN2): now also J1.3 (Pin_3)
- no-connect marks 8 -> 12
Other:
- note added: "PC RXD"
- note added: "PC TXD"
- moved on the sheet: U2
