File: hardware/schematic/v1.0/CORE/CORE.kicad_sch (KiCad schematic)
At the start: 47 parts, among them J1 Conn_01x03_Socket, M1 ZYNQ7010&7020, U1 TXS02612RTWR, U2 SP3232, U3 SD_Card

Commit message: sch update
Parts:
- added J2, J3, J4, J5: Conn_Coaxial, Connector_Coaxial:SMA_Amphenol_132289_EdgeMount, symbol Connector:Conn_Coaxial
- added R24, R25, R26, R27: 0, Resistor_SMD:R_0402_1005Metric, symbol Device:R
Connections:
- net GND: now also J2.2 (Ext), J3.2 (Ext), J4.2 (Ext), J5.2 (Ext)
- new net: J4.1 (In), R26.1
- new net: J5.1 (In), R27.1
- new net: J3.1 (In), R25.1
- new net: J2.1 (In), R24.1
- new net CLK_FS_N: R27.2
- new net CLK_FS_P: R26.2
- new net CLK_FX_N: R25.2
- new net CLK_FX_P: R24.2

Commit message: sch update
Parts:
- added J6, J7, J8, J9: Conn_Coaxial, Connector_Coaxial:SMA_Amphenol_132289_EdgeMount, symbol Connector:Conn_Coaxial
- added R28, R29, R30, R31, R32, R33: 0, Resistor_SMD:R_0402_1005Metric, symbol Device:R
Connections:
- net CLK_FS_N: now also R32.2
- net CLK_FS_P: now also R33.2
- net CLK_FX_N: now also M1.J2_36 (36)
- net CLK_FX_P: now also M1.J2_34 (34)
- net GND: now also M1.J1_100 (100), M1.J1_93 (93), M1.J1_94 (94), M1.J1_95 (95), M1.J1_96 (96), M1.J1_97 (97), M1.J1_98 (98), M1.J1_99 (99), J6.2 (Ext), J7.2 (Ext), J8.2 (Ext), J9.2 (Ext)
- net at M1.J1_65 (65): now also R32.1
- net at M1.J1_67 (67): now also R33.1
- new net: J8.1 (In), R30.1
- new net: J7.1 (In), R29.1
- new net: J9.1 (In), R31.1
- new net: J6.1 (In), R28.1
- new net CLK1_FS_N: R31.2
- new net CLK1_FS_P: R30.2
- new net CLK1_FX_N: R29.2
- new net CLK1_FX_P: R28.2
Other:
- note added: "B35_L2_N_A20"
- note added: "B35_L2_P_B19"
- note added: "ETHERNET(PS)"
- note added: "JTAG"
- note added: "PS/PL LED"
- note added: "RS232"
- note added: "SD_CARD"
- note added: "SIGNAL"
- moved on the sheet: BOOT_CFG, C10, C2, C3, C4, C5, C6, C7, C8, C9, D3, D4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

Commit message: sch update
Parts:
- added C11, C15: 4.7uF, Capacitor_SMD:C_0603_1608Metric, symbol Device:C
- added C12, C14, C16, C18: 100nF, Capacitor_SMD:C_0603_1608Metric, symbol Device:C
- added C13, C17: 10uF, Capacitor_SMD:C_0603_1608Metric, symbol Device:C
- added J10: USB_C_Receptacle_USB2.0_16P, symbol Connector:USB_C_Receptacle_USB2.0_16P
- added U4: AMS1117-2.5, Package_TO_SOT_SMD:SOT-223-3_TabPin2, symbol Regulator_Linear:AMS1117-2.5
- added U5: AMS1117-1.8, Package_TO_SOT_SMD:SOT-223-3_TabPin2, symbol Regulator_Linear:AMS1117-1.8
Connections:
- net +1.8V: now also C17.1, C18.1, U5.2 (VO)
- net +5V: now also C11.1, C12.1, C15.1, C16.1, U4.3 (VI), U5.3 (VI)
- net GND: now also C11.2, C12.2, C13.2, C14.2, C15.2, C16.2, C17.2, C18.2, U4.1 (GND), U5.1 (GND)
- new net: J10.A1 (GND), J10.A12 (GND), J10.B1 (GND), J10.B12 (GND)
- new net: J10.A4 (VBUS), J10.A9 (VBUS), J10.B4 (VBUS), J10.B9 (VBUS)
- new net +2.5V: C13.1, C14.1, U4.2 (VO)
Other:
- moved on the sheet: BOOT_CFG, C1, C10, C2, C3, C4, C5, C6, C7, C8, C9, D1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

Commit message: sch update
Parts:
- added J11: Conn_01x06_Socket, Connector_PinSocket_2.54mm:PinSocket_1x06_P2.54mm_Vertical, symbol Connector:Conn_01x06_Socket
Connections:
- net CLK1_FX_N: now also M1.J2_38 (38)
- net CLK1_FX_P: now also M1.J2_40 (40)
- net CLK_FX_N: now also M1.J2_26 (26); no longer M1.J2_36 (36)
- net CLK_FX_P: now also M1.J2_28 (28); no longer M1.J2_34 (34)
- net PS_I2C_SDA: no longer M1.J2_65 (65)
- new net PS_I2C_SCL: M1.J2_65 (65)
Other:
- note added: "MRCC B34_L13_N P19"
- note added: "MRCC B34_L13_P N18"
- note added: "MRCC B35_L12_N K18"
- note added: "MRCC B35_L12_P K17"
- note added: "MRCC B35_L13_N H17"
- note added: "MRCC B35_L13_P H16"
- note added: "PS_MIO30"
- note added: "PS_MIO31"
- note added: "SRCC B34_L14_N P20"
- note added: "SRCC B34_L14_P N20"
- note added: "SRCC B35_L11_N L17"
- note added: "SRCC B35_L11_P L16"
- note added: "SRCC B35_L14_N H18"
- note added: "SRCC B35_L14_P J18"

Commit message: sch update
Parts:
- C5: value 10uF -> 100nF
Connections:
- net GND: now also M1.J1_19 (19), M1.J1_34 (34), M1.J1_41 (41), M1.J1_52 (52), M1.J1_59 (59), M1.J1_70 (70), M1.J2_11 (11), M1.J2_12 (12), M1.J2_62 (62), M1.J2_63 (63), M1.J2_76 (76), M1.J2_77 (77)
- net PHY1_AD0/LED0: now reaches M1.J2_1 (1)
- net PHY1_AD0/LED0: now also GE_PS1.12 (GC)
- net PHY1_MDI3_N: now reaches M1.J2_10 (10)
- net PHY1_MDI3_N: now also D2.5 (Line-4)
- net PHY1_AD1/LED1: now reaches M1.J2_2 (2)
- net PHY1_AD1/LED1: now also GE_PS1.13 (YC)
- net PHY1_MDI0_P: now reaches M1.J2_3 (3)
- net PHY1_MDI0_P: now also D1.1 (Line-1)
- net PHY1_MDI2_P: now reaches M1.J2_4 (4)
- net PHY1_MDI2_P: now also D2.1 (Line-1)
- net PHY1_MDI0_N: now reaches M1.J2_5 (5)
- net PHY1_MDI0_N: now also D1.2 (Line-2)
- net PHY1_MDI2_N: now reaches M1.J2_6 (6)
- net PHY1_MDI2_N: now also D2.2 (Line-2)
- net PHY1_MDI1_P: now reaches M1.J2_7 (7)
- net PHY1_MDI1_P: now also D1.4 (Line-3)
- net PHY1_MDI3_P: now reaches M1.J2_8 (8)
- net PHY1_MDI3_P: now also D2.4 (Line-3)
- net PHY1_MDI1_N: now reaches M1.J2_9 (9)
- net PHY1_MDI1_N: now also D1.5 (Line-4)
Other:
- moved on the sheet: R9

Commit message: sch update
Parts:
- added R34, R35: 0, Resistor_SMD:R_0402_1005Metric, symbol Device:R
Connections:
- net CLK1_FS_N: now also M1.J1_14 (14)
- net CLK1_FS_P: now also M1.J1_12 (12)
- net CLK_FS_N: now also M1.J1_18 (18)
- net CLK_FS_P: now also M1.J1_16 (16)
- net GND: now also J11.1 (Pin_1)
- net PS_I2C_SCL: now also J11.3 (Pin_3)
- net PS_I2C_SDA: now also J11.2 (Pin_2)
- net at M1.J1_53 (53): now also R34.1
- net at M1.J1_55 (55): now also R35.1
- new net STATUS0: R34.2
- new net STATUS1: R35.2
Other:
- moved on the sheet: J10

Commit message: sch update
Parts:
- removed J1: Conn_01x03_Socket, Connector_PinHeader_2.54mm:PinHeader_1x03_P2.54mm_Vertical, symbol Connector:Conn_01x03_Socket
- removed R34, R35: 0, Resistor_SMD:R_0402_1005Metric, symbol Device:R
- removed U2: SP3232, Counter:SOP16M, symbol Counter:MAX3232
- added C19, C22: 100nF, Capacitor_SMD:C_0402_1005Metric, symbol Device:C
- added C20: 2.2uF, Capacitor_SMD:C_0402_1005Metric, symbol Device:C
- added C21: 10nF, Capacitor_SMD:C_0402_1005Metric, symbol Device:C
- added C23: 1uF, Capacitor_SMD:C_0402_1005Metric, symbol Device:C
- added J1: Conn_01x16_Socket, Connector_PinSocket_2.54mm:PinSocket_1x16_P2.54mm_Vertical, symbol Connector:Conn_01x16_Socket
- added R36, R37: 5.1K, Resistor_SMD:R_0402_1005Metric, symbol Device:R
- added R38, R39, R40, R41: 0, Resistor_SMD:R_0402_1005Metric, symbol Device:R
- added U2, U7: TPS78633, Package_TO_SOT_SMD:SOT-223-6, symbol Counter:TPS78633
- added U6: CH340E, Package_SO:MSOP-10_3x3mm_P0.5mm, symbol Interface_USB:CH340E
- C10: value 100nF -> 1uF
- C7: value 100nF -> 10uF
- C8: value 100nF -> 2.2uF
- C9: value 100nF -> 10nF
Connections:
- net +3.3V: now also C10.2, C19.2, C22.2, C23.2, J1.3 (Pin_3), J1.4 (Pin_4), U2.4 (OUT), U6.10 (V3), U6.7 (VCC), U7.4 (OUT); no longer C6.2, C7.2
- net +5V: now also C6.1, C7.1, J10.A4 (VBUS), J10.A9 (VBUS), J10.B4 (VBUS), J10.B9 (VBUS), J1.1 (Pin_1), J1.2 (Pin_2), R40.2, R41.2, U2.2 (IN), U7.2 (IN)
- net GND: now also C10.1, C6.2, C7.2, C8.1, C9.1, J10.A1 (GND), J10.A12 (GND), J10.B1 (GND), J10.B12 (GND), J10.SH (SHIELD), C19.1, C20.1, C21.1, C22.1, C23.1, J1.5 (Pin_5), J1.6 (Pin_6), R36.2, R37.1, U2.3 (GND), U2.6 (TAB), U6.3 (GND), U7.3 (GND), U7.6 (TAB); no longer C10.2, C7.1
- net PS_I2C_SCL: no longer M1.J2_65 (65)
- net PS_I2C_SDA: no longer M1.J2_70 (70)
- net IO0: now reaches M1.J1_43 (43)
- net IO0: now also J1.9 (Pin_9)
- net IO1: now reaches M1.J1_45 (45)
- net IO1: now also J1.10 (Pin_10)
- net IO2: now reaches M1.J1_47 (47)
- net IO2: now also J1.11 (Pin_11)
- net IO3: now reaches M1.J1_49 (49)
- net IO3: now also J1.12 (Pin_12)
- net IO4: now reaches M1.J1_51 (51)
- net IO5: now reaches M1.J1_53 (53)
- net IO5: now also J1.13 (Pin_13)
- net IO6: now reaches M1.J1_55 (55)
- net IO6: now also J1.14 (Pin_14)
- net IO7: now reaches M1.J1_57 (57)
- net at C8.2: now also R40.1, U2.1 (EN)
- net at J10.A5 (CC1): now also R36.1
- net USB_D+: now reaches J10.A6 (D+)
- net USB_D+: now also J10.B6 (D+), U6.1 (UD+)
- net USB_D-: now reaches J10.A7 (D-)
- net USB_D-: now also J10.B7 (D-), U6.2 (UD-)
- net at J10.B5 (CC2): now also R37.2
- net at C9.2: now also U2.5 (NR/FB)
- net PS_UART1_RXD renamed RXD
- net RXD: now also R38.2
- net PS_UART1_TXD renamed TXD
- net TXD: now also R39.1
- new net: C20.2, R41.1, U7.1 (EN)
- new net: R38.1, U6.8 (TXD)
- new net: R39.2, U6.9 (RXD)
- new net: C21.2, U7.5 (NR/FB)
- new net I2C_SCL: J1.8 (Pin_8), M1.J2_65 (65)
- new net I2C_SDA: J1.7 (Pin_7), M1.J2_70 (70)
- no-connect marks 12 -> 13
Other:
- note added: "POWER"
- note added: "SOCKET"
- note removed: "PC RXD"
- note removed: "PC TXD"
- note removed: "RS232"
- moved on the sheet: C11, C12, C13, C14, C15, C16, C17, C18, J10, U4, U5

Commit message: shc update
Parts:
- removed R32, R33: 0, Resistor_SMD:R_0402_1005Metric, symbol Device:R
- D3, D4, D5, D6: footprint (none) -> LED_SMD:LED_0603_1608Metric
- J10: footprint (none) -> Connector_USB:USB_C_Receptacle_Palconn_UTC16-G
- U3: footprint (none) -> Counter:SIM-SMD_LX_XDFP-0090-012
- renumbered BOOT_CFG to BOOT_CFG1
Connections:
- net CLK1_FS_N: now also M1.J1_48 (48); no longer M1.J1_14 (14)
- net CLK1_FS_P: now also M1.J1_50 (50); no longer M1.J1_12 (12)
Other:
- note added: "SRCC B34_L11_N U15"
- note added: "SRCC B34_L11_P U14"
- moved on the sheet: J6, J7, R28, R29
