File: hardware/schematic/v1.0/CORE/CORE.kicad_pcb (KiCad board)
At the start: 2 copper layers, 1 x 9 mm, 88 parts, among them J1 Conn_01x16_Socket, J10 USB_C_Receptacle_USB2.0_16P, J11 Conn_01x06_Socket, J2 Conn_Coaxial, J3 Conn_Coaxial, J4 Conn_Coaxial, J5 Conn_Coaxial, J6 Conn_Coaxial, J7 Conn_Coaxial, J8 Conn_Coaxial, J9 Conn_Coaxial, M1 ZYNQ7010&7020, U1 TXS02612RTWR, U2 TPS78633, U3 SD_Card, U4 AMS1117-2.5, U5 AMS1117-1.8, U6 CH340E, U7 TPS78633

Commit message: sch update
Connections:
- M1 pad J2_90: unconnected-(M1-90-PadJ2_90) -> SPI1_SCLK
- M1 pad J2_91: SD_CD -> SPI1_MOSI
- M1 pad J2_93: unconnected-(M1-93-PadJ2_93) -> SPI1_SS0
- M1 pad J2_94: unconnected-(M1-94-PadJ2_94) -> SPI1_MISO
Changed lines of the file:
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@@
 			(size 1.7 0.35001)
 			(layers "F.Cu" "F.Mask" "F.Paste")
-			(net "unconnected-(M1-90-PadJ2_90)")
+			(net "SPI1_SCLK")
 			(pinfunction "90_J2_90")
 			(pintype "passive")
@@
 			(size 1.7 0.35001)
 			(layers "F.Cu" "F.Mask" "F.Paste")
-			(net "SD_CD")
+			(net "SPI1_MOSI")
 			(pinfunction "91_J2_91")
 			(pintype "passive")
@@
 			(size 1.7 0.35001)
 			(layers "F.Cu" "F.Mask" "F.Paste")
-			(net "unconnected-(M1-93-PadJ2_93)")
+			(net "SPI1_SS0")
 			(pinfunction "93_J2_93")
 			(pintype "passive")
@@
 			(size 1.7 0.35001)
 			(layers "F.Cu" "F.Mask" "F.Paste")
-			(net "unconnected-(M1-94-PadJ2_94)")
+			(net "SPI1_MISO")
 			(pinfunction "94_J2_94")
 			(pintype "passive")

Commit message: sch update
Parts:
- added J12: Conn_01x16_Socket, Connector_PinSocket_2.54mm:PinSocket_1x16_P2.54mm_Vertical, F.Cu at (169.3, 37.8)
Connections:
- M1 pad J2_96: unconnected-(M1-96-PadJ2_96) -> SD_CD

Commit message: sch update
Parts:
- C10, C23: value 1uF -> 10uF; footprint Capacitor_SMD:C_0402_1005Metric -> Capacitor_SMD:C_0603_1608Metric
- C11, C15: value 4.7uF -> 10uF
- C20, C8: value 2.2uF -> 10uF; footprint Capacitor_SMD:C_0402_1005Metric -> Capacitor_SMD:C_0603_1608Metric
- moved C10 71.8 mm to (195.0, 49.2), turned to -90 degrees
- moved C9 69.7 mm to (198.0, 51.5), turned to 90 degrees
- moved C21 68.8 mm to (209.5, 66.8), turned to 90 degrees
- moved C19 68.8 mm to (197.8, 49.2), turned to -90 degrees
- moved C23 68.3 mm to (206.8, 64.2), turned to -90 degrees
- moved C22 67.0 mm to (209.2, 64.5), turned to -90 degrees
- moved C8 65.8 mm to (200.8, 43.5), turned to 180 degrees
- moved C15 56.7 mm to (238.0, 111.2)
- moved C16 56.3 mm to (238.0, 113.2)
- moved C20 56.2 mm to (212.2, 58.5), turned to 180 degrees
- moved R40 51.5 mm to (197.2, 46.5), turned to -90 degrees
- moved U5 47.9 mm to (240.3, 106.0)
- moved C11 46.4 mm to (240.2, 91.0)
- moved R41 43.5 mm to (209.0, 61.8), turned to -90 degrees
- moved C17 43.4 mm to (246.5, 105.0), turned to 90 degrees
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Connections:
- C11 pad 1: +5V -> +3.3V
- C12 pad 1: +5V -> +3.3V
- C15 pad 1: +5V -> +3.3V
- C16 pad 1: +5V -> +3.3V
- M1 pad J2_83: unconnected-(M1-83-PadJ2_83) -> XADC_VP
- M1 pad J2_85: unconnected-(M1-85-PadJ2_85) -> XADC_VN
- U4 pad 3: +5V -> +3.3V
- U5 pad 3: +5V -> +3.3V

Commit message: sch update
Parts:
- removed J12: Conn_01x16_Socket, Connector_PinSocket_2.54mm:PinSocket_1x16_P2.54mm_Vertical
- added J13: Conn_01x10_Socket, Connector_PinHeader_2.54mm:PinHeader_1x10_P2.54mm_Vertical, F.Cu at (157.9, 139.8)
- added J14: Conn_01x10_Socket, Connector_PinHeader_2.54mm:PinHeader_1x10_P2.54mm_Vertical, F.Cu at (97.3, 48.5)
- C7: footprint Capacitor_SMD:C_0402_1005Metric -> Capacitor_SMD:C_0603_1608Metric
- J1: value Conn_01x16_Socket -> Conn_01x06_Socket; footprint Connector_PinSocket_2.54mm:PinSocket_1x16_P2.54mm_Vertical -> Connector_PinHeader_2.54mm:PinHeader_1x06_P2.54mm_Vertical
- J11: footprint Connector_PinSocket_2.54mm:PinSocket_1x06_P2.54mm_Vertical -> Connector_PinHeader_2.54mm:PinHeader_1x06_P2.54mm_Vertical
- moved J4 92.4 mm to (74.0, 98.3), turned to 180 degrees
- moved J11 84.9 mm to (176.7, 48.4), turned to -90 degrees
- moved R26 82.8 mm to (81.1, 98.3), turned to 0 degrees
- moved J5 73.9 mm to (74.0, 114.2), turned to 180 degrees
- moved C6 65.1 mm to (179.2, 65.7)
- moved U6 65.1 mm to (176.2, 60.3)
- moved J10 65.1 mm to (183.9, 60.4)
- moved R38 65.1 mm to (177.2, 55.2)
- moved R39 65.1 mm to (175.7, 55.2)
- moved R36 65.1 mm to (184.7, 67.7)
- moved R37 65.1 mm to (184.7, 53.2)
- moved C7 64.5 mm to (177.7, 66.2)
- moved R27 64.4 mm to (81.2, 114.2), turned to 0 degrees
- moved U7 51.0 mm to (164.5, 71.8), turned to 180 degrees
- moved C20 48.8 mm to (167.1, 77.0), turned to 0 degrees
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Connections:
- J11 pad 1: GND -> +5V
- J11 pad 2: PS_I2C_SDA -> +5V
- J11 pad 3: PS_I2C_SCL -> +3.3V
- J11 pad 4: unconnected-(J11-Pin_4-Pad4) -> +3.3V
- J11 pad 5: unconnected-(J11-Pin_5-Pad5) -> GND
- J11 pad 6: unconnected-(J11-Pin_6-Pad6) -> GND
Routing:
- net CLK_FX_N: track 0.00 -> 25.8 mm
- net CLK_FX_P: track 0.00 -> 25.7 mm
- net Net-(J2-In): track 0.00 -> 5.64 mm
- net Net-(J3-In): track 0.00 -> 5.49 mm
- net Net-(JTAG1-Pad10): track 0.00 -> 5.47 mm
- net Net-(JTAG1-Pad8): track 0.00 -> 5.47 mm
- net Net-(JTAG1-Pad6): track 0.00 -> 5.47 mm
- net Net-(JTAG1-Pad4): track 0.00 -> 5.46 mm
- net Net-(BOOT_CFG1-Pad4): track 0.00 -> 3.18 mm
- net Net-(BOOT_CFG1-Pad3): track 0.00 -> 3.16 mm
- net Net-(D4-A): track 0.00 -> 1.86 mm
- net Net-(D3-A): track 0.00 -> 1.82 mm
Other:
- board size 1 x 9 mm -> 118 x 97 mm

Commit message: sch update
Parts:
- removed C13, C20, C23: 10uF, Capacitor_SMD:C_0603_1608Metric
- removed C14: 100nF, Capacitor_SMD:C_0603_1608Metric
- removed C21: 10nF, Capacitor_SMD:C_0402_1005Metric
- removed C22: 100nF, Capacitor_SMD:C_0402_1005Metric
- removed R24, R25, R28, R29, R30, R31, R41: 0, Resistor_SMD:R_0402_1005Metric
- removed U4: AMS1117-2.5, Package_TO_SOT_SMD:SOT-223-3_TabPin2
- removed U7: TPS78633, Package_TO_SOT_SMD:SOT-223-6
- C11: value 10uF -> 100nF; footprint Capacitor_SMD:C_0603_1608Metric -> Capacitor_SMD:C_0402_1005Metric
- C12: value 100nF -> 10uF
- moved U5 78.8 mm to (167.8, 75.3), turned to -90 degrees
- moved C17 78.1 mm to (173.1, 78.2)
- moved C16 78.1 mm to (166.5, 69.7), turned to 0 degrees
- moved C18 78.1 mm to (175.2, 78.2)
- moved C15 77.4 mm to (166.5, 67.7), turned to 0 degrees
- moved C12 65.5 mm to (181.1, 50.9), turned to 180 degrees
- moved C11 63.1 mm to (181.2, 52.5), turned to 180 degrees
- moved J14 24.3 mm to (87.3, 26.3)
- moved J4 3.80 mm to (73.9, 94.5)
- moved J5 3.80 mm to (74.0, 110.4)
- moved R26 3.80 mm to (81.0, 94.5)
- moved R27 3.80 mm to (81.1, 110.4)
- moved U3 3.31 mm to (81.4, 72.3)
- moved R16 3.31 mm to (88.2, 61.7)
- moved R17 3.31 mm to (88.2, 59.2)
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Connections:
- C11 pad 1: +3.3V -> +5V
- C12 pad 1: +3.3V -> +5V
- J2 pad 1: Net-(J2-In) -> CLK_FX_P
- J3 pad 1: Net-(J3-In) -> CLK_FX_N
- J4 pad 1: Net-(J4-In) -> CLK_FS_P
- J5 pad 1: Net-(J5-In) -> CLK_FS_N
- J6 pad 1: Net-(J6-In) -> CLK1_FX_P
- J7 pad 1: Net-(J7-In) -> CLK1_FX_N
- J8 pad 1: Net-(J8-In) -> CLK1_FS_P
- J9 pad 1: Net-(J9-In) -> CLK1_FS_N
Routing:
- net CLK_FX_N: track 25.8 -> 0.00 mm
- net CLK_FX_P: track 25.7 -> 0.00 mm
- net Net-(J2-In): track 5.64 -> 0.00 mm
- net Net-(J3-In): track 5.49 -> 0.00 mm
- added copper zone on In2.Cu, net +1.8V
- added copper zone on In2.Cu, net +3.3V
- added copper zone on In2.Cu, net +5V
- added copper zone on In1.Cu, net GND
Other:
- copper layers 2 -> 4

Commit message: core update
Parts:
- removed R26, R27: 0, Resistor_SMD:R_0402_1005Metric
- added J12: Conn_Coaxial, Connector_Coaxial:SMA_Amphenol_132289_EdgeMount, F.Cu at (74.3, 131.0)
- added J15: Conn_01x05_Socket, Connector_PinHeader_2.54mm:PinHeader_1x05_P2.54mm_Vertical, F.Cu at (77.8, 48.6)
- added J16: Conn_01x04_Socket, Connector_PinHeader_2.54mm:PinHeader_1x04_P2.54mm_Vertical, F.Cu at (136.8, 126.7)
- J13: value Conn_01x10_Socket -> Conn_01x04_Socket; footprint Connector_PinHeader_2.54mm:PinHeader_1x10_P2.54mm_Vertical -> Connector_PinHeader_2.54mm:PinHeader_1x04_P2.54mm_Vertical
- J14: value Conn_01x10_Socket -> Conn_01x03_Socket; footprint Connector_PinHeader_2.54mm:PinHeader_1x10_P2.54mm_Vertical -> Connector_PinHeader_2.54mm:PinHeader_1x03_P2.54mm_Vertical
- moved J14 103.8 mm to (91.2, 130.0), turned to 0 degrees
- moved J1 73.6 mm to (157.4, 136.8), turned to -90 degrees
- moved J13 20.4 mm to (138.3, 134.2)
- moved C18 13.9 mm to (161.2, 78.2)
- moved C17 10.1 mm to (163.0, 78.2)
- moved D6 4.89 mm to (90.7, 88.4)
- moved R7 4.89 mm to (95.3, 84.8)
- moved R8 4.89 mm to (95.3, 88.2)
- moved D5 4.89 mm to (90.7, 84.8)
- moved J6 3.65 mm to (104.1, 47.0)
- moved C3 1.36 mm to (108.3, 66.0)
Connections:
- J13 pad 1: I2C_SDA -> IO0
- J13 pad 2: I2C_SCL -> IO1
- J13 pad 3: IO0 -> IO2
- J13 pad 4: IO1 -> IO3
- J14 pad 1: SPI1_MOSI -> I2C_SDA
- J14 pad 2: SPI1_MISO -> I2C_SCL
- J14 pad 3: SPI1_SCLK -> GND
Routing:
- net +1.8V: track 0.00 -> 3.85 mm

Commit message: sch update
Parts:
- added C13: 1nF, Capacitor_SMD:C_0402_1005Metric, F.Cu at (34.4, 132.0)
- added J26: Conn_01x04_Socket, Connector_PinHeader_2.54mm:PinHeader_1x04_P2.54mm_Vertical, F.Cu at (30.7, 129.3)
- added R41: 49.9, Resistor_SMD:R_0402_1005Metric, F.Cu at (34.4, 128.0)
- added R42: 49.9, Resistor_SMD:R_0402_1005Metric, F.Cu at (34.4, 130.0)
- added RGB TFTLCD1: RGBLCD, AD:FPC-TOP40, B.Cu at (91.5, 88.7)
- moved J8 18.3 mm to (125.3, 138.7)
- moved J9 8.55 mm to (110.8, 138.7)
- moved D5 6.62 mm to (92.0, 78.3)
- moved D6 6.62 mm to (92.0, 81.9)
- moved R7 6.62 mm to (96.6, 78.2)
- moved R8 6.62 mm to (96.6, 81.8)
- moved J13 5.37 mm to (143.2, 132.0)
- moved J4 0.65 mm to (73.9, 93.8)
- moved J5 0.65 mm to (74.0, 109.8)
Connections:
- net I2C_SCL renamed PS_I2C_SCL
- net I2C_SDA renamed PS_I2C_SDA
- net SPI1_MISO renamed PS_SPI1_MISO
- net SPI1_MOSI renamed PS_SPI1_MOSI
- net SPI1_SCLK renamed PS_SPI1_SCLK
- net SPI1_SS0 renamed PS_SPI1_SS0
- M1 pad J1_48: CLK1_FS_N -> unconnected-(M1-48-PadJ1_48)
- M1 pad J1_50: CLK1_FS_P -> unconnected-(M1-50-PadJ1_50)
- M1 pad J1_81: unconnected-(M1-81-PadJ1_81) -> CLK1_FS_P
- M1 pad J1_83: unconnected-(M1-83-PadJ1_83) -> CLK1_FS_N

Commit message: sch update
Parts:
- removed J12, J6, J7, J8, J9: Conn_Coaxial, Connector_Coaxial:SMA_Amphenol_132289_EdgeMount
- added U10: IPEX1, Counter:JLC_IPEX-1, F.Cu at (119.3, 138.8)
- added U11: IPEX1, Counter:JLC_IPEX-1, F.Cu at (114.8, 138.8)
- added U4: IPEX1, Counter:JLC_IPEX-1, F.Cu at (127.7, 139.1)
- added U8: IPEX1, Counter:JLC_IPEX-1, F.Cu at (112.9, 46.9)
- added U9: IPEX1, Counter:JLC_IPEX-1, F.Cu at (118.9, 46.9)
- moved J2 3.85 mm to (130.9, 47.0)
- moved J3 3.85 mm to (147.1, 47.0)
- moved J4 0.11 mm to (74.0, 93.9)
- moved J5 0.11 mm to (74.0, 109.8)
Connections:
- M1 pad J1_25: unconnected-(M1-25-PadJ1_25) -> LCD_R2
- M1 pad J1_26: unconnected-(M1-26-PadJ1_26) -> LCD_R0
- M1 pad J1_27: unconnected-(M1-27-PadJ1_27) -> LCD_R3
- M1 pad J1_28: unconnected-(M1-28-PadJ1_28) -> LCD_R1
- M1 pad J1_29: unconnected-(M1-29-PadJ1_29) -> LCD_R6
- M1 pad J1_30: unconnected-(M1-30-PadJ1_30) -> LCD_R4
- M1 pad J1_31: unconnected-(M1-31-PadJ1_31) -> LCD_R7
- M1 pad J1_32: unconnected-(M1-32-PadJ1_32) -> LCD_R5
- M1 pad J1_33: unconnected-(M1-33-PadJ1_33) -> LCD_G0
- M1 pad J1_35: unconnected-(M1-35-PadJ1_35) -> LCD_G1
- M1 pad J1_36: unconnected-(M1-36-PadJ1_36) -> LCD_G2
- M1 pad J1_37: unconnected-(M1-37-PadJ1_37) -> LCD_G4
- M1 pad J1_38: unconnected-(M1-38-PadJ1_38) -> LCD_G3
- M1 pad J1_39: unconnected-(M1-39-PadJ1_39) -> LCD_G5
- M1 pad J1_40: unconnected-(M1-40-PadJ1_40) -> LCD_G6
- M1 pad J1_42: unconnected-(M1-42-PadJ1_42) -> LCD_G7
- M1 pad J1_43: IO0 -> LCD_B2
- M1 pad J1_44: unconnected-(M1-44-PadJ1_44) -> LCD_B0
- M1 pad J1_45: IO1 -> LCD_B3
- M1 pad J1_46: unconnected-(M1-46-PadJ1_46) -> LCD_B1
- M1 pad J1_47: IO2 -> LCD_B6
- M1 pad J1_48: unconnected-(M1-48-PadJ1_48) -> LCD_B4
- M1 pad J1_49: IO3 -> LCD_B7
- M1 pad J1_50: unconnected-(M1-50-PadJ1_50) -> LCD_B5
- M1 pad J1_51: IO4 -> CTP_RST
- M1 pad J1_53: IO5 -> CTP_INT
- M1 pad J1_54: unconnected-(M1-54-PadJ1_54) -> LCD_CLK
- M1 pad J1_55: IO6 -> CTP_SDA
- M1 pad J1_56: unconnected-(M1-56-PadJ1_56) -> LCD_DISP
- M1 pad J1_57: IO7 -> CTP_SCL
- M1 pad J1_58: unconnected-(M1-58-PadJ1_58) -> LCD_HSYNC
- M1 pad J1_60: unconnected-(M1-60-PadJ1_60) -> LCD_VSYNC
- M1 pad J1_62: unconnected-(M1-62-PadJ1_62) -> LCD_DE
- M1 pad J1_77: unconnected-(M1-77-PadJ1_77) -> CLK_10M
- RGB TFTLCD1 pad 1: unconnected-(RGB TFTLCD1-Pad1) -> LCD_LEDK
- RGB TFTLCD1 pad 2: unconnected-(RGB TFTLCD1-Pad2) -> LCD_LEDA
