File: hardware/schematic/v1.0/CORE/ZynqCore.kicad_sch (KiCad schematic)
At the start: 1 part, among them M1 ZYNQ7010&7020

Commit message: sch update
Connections:
- net LCD_BLK: now reaches M1.J1_24 (24)
Changed lines of the file:
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@@
 	(polyline
 		(pts
-			(xy 44.45 17.78) (xy 247.65 17.78)
+			(xy 43.18 17.78) (xy 247.65 17.78)
 		)
 		(stroke
@@
 	(polyline
 		(pts
-			(xy 44.45 17.78) (xy 44.45 163.83)
+			(xy 43.18 17.78) (xy 43.18 163.83)
 		)
 		(stroke
@@
 		)
 	)
-	(hierarchical_label "LCD_LEDA"
-		(shape output)
-		(at 31.75 57.15 0)
-		(effects
-			(font
-				(size 1.27 1.27)
-			)
-			(justify left)
-		)
-	)
 	(hierarchical_label "CTP_SDA"
 		(shape output)
@@
 		)
 	)
-	(hierarchical_label "LCD_LEDK"
+	(hierarchical_label "LCD_BLK"
 		(shape output)
-		(at 31.75 54.61 0)
-		(effects
-			(font
-				(size 1.27 1.27)
-			)
-			(justify left)
-		)
-	)
+		(at 62.23 59.69 180)
+		(effects
+			(font
+				(size 1.27 1.27)
+			)
+			(justify right)
+		)
+	)

Commit message: sch update
Connections:
- net CLK_FS_N is gone; now on net CLK1_FS_N: M1.J1_18 (18)
- net CLK_FS_P is gone; now on net CLK1_FS_P: M1.J1_16 (16)
- net CLK1_FS_N: no longer M1.J1_83 (83)
- net CLK1_FS_P: no longer M1.J1_81 (81)
- net CLK1_FX_N: no longer M1.J2_38 (38)
- net CLK1_FX_P: no longer M1.J2_40 (40)
- net CLK_FX_N: no longer names the net of M1.J2_26 (26)
- net CLK_FX_P: no longer names the net of M1.J2_28 (28)
- new net CLK2_FS_N: M1.J1_83 (83)
- new net CLK2_FS_P: M1.J1_81 (81)
