File: hardware/schematic/v1.0/CORE/ZynqCore.kicad_sch (KiCad schematic)
At the start: 1 part, among them M1 ZYNQ7010&7020

Commit message: sch update
Connections:
- net CLK1_FX_N: now also M1.J2_18 (18)
- net CLK1_FX_P: now also M1.J2_20 (20)
- net CLK2_FX_N: now also M1.J2_26 (26)
- net CLK2_FX_P: now also M1.J2_28 (28)
- net CLK3_FX_N: now also M1.J2_38 (38)
- net CLK3_FX_P: now also M1.J2_40 (40)
- net CLK4_FX_N: now also M1.J2_50 (50)
- net CLK4_FX_P: now also M1.J2_52 (52)
- net CLK5_FX_N: now also M1.J2_58 (58)
- net CLK5_FX_P: now also M1.J2_60 (60)
- net CLK6_FX_N: now also M1.J2_19 (19)
- net CLK6_FX_P: now also M1.J2_17 (17)
- net CLK7_FX_N: now also M1.J2_27 (27)
- net CLK7_FX_P: now also M1.J2_25 (25)
- net CLK8_FX_N: now also M1.J2_35 (35)
- net CLK8_FX_P: now also M1.J2_33 (33)
- no-connect marks 10 -> 4
Changed lines of the file:
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@@
-	)
-	(no_connect
-		(at 163.83 72.39)
-	)
-	(no_connect
-		(at 223.52 64.77)
-	)
-	(no_connect
-		(at 163.83 74.93)
 	)
 	(no_connect
@@
 	)
 	(no_connect
-		(at 223.52 62.23)
-	)
-	(no_connect
-		(at 163.83 95.25)
-	)
-	(no_connect
 		(at 62.23 44.45)
 	)
@@
 	)
 	(no_connect
-		(at 163.83 92.71)
-	)
-	(no_connect
 		(at 77.47 146.05)
 	)
@@
 		)
 	)
+	(hierarchical_label "CLK5_FX_N"
+		(shape input)
+		(at 163.83 102.87 180)
+		(effects
+			(font
+				(size 1.27 1.27)
+			)
+			(justify right)
+		)
+	)
 	(hierarchical_label "LCD_R6"
 		(shape output)
@@
 		)
 	)
+	(hierarchical_label "CLK4_FX_P"
+		(shape input)
+		(at 163.83 95.25 180)
+		(effects
+			(font
+				(size 1.27 1.27)
+			)
+			(justify right)
+		)
+	)
 	(hierarchical_label "CLK2_FX_N"
 		(shape input)
-		(at 270.51 62.23 180)
+		(at 163.83 62.23 180)
 		(effects
 			(font
@@
 		)
 	)
-	(hierarchical_label "CLK5_FX_N"
-		(shape input)
-		(at 270.51 85.09 180)
-		(effects
-			(font
-				(size 1.27 1.27)
-			)
-			(justify right)
-		)
-	)
 	(hierarchical_label "LCD_R2"
 		(shape output)
@@
 		)
 	)
-	(hierarchical_label "CLK4_FX_N"
-		(shape input)
-		(at 270.51 77.47 180)
-		(effects
-			(font
-				(size 1.27 1.27)
-			)
-			(justify right)
-		)
-	)
 	(hierarchical_label "LCD_CLK"
 		(shape output)
@@
 		)
 	)
+	(hierarchical_label "CLK5_FX_P"
+		(shape input)
+		(at 163.83 105.41 180)
+		(effects
+			(font
+				(size 1.27 1.27)
+			)
+			(justify right)
+		)
+	)
 	(hierarchical_label "CLK8_FX_N"
 		(shape input)
-		(at 270.51 107.95 180)
-		(effects
-			(font
-				(size 1.27 1.27)
-			)
-			(justify right)
+		(at 223.52 74.93 0)
+		(effects
+			(font
+				(size 1.27 1.27)
+			)
+			(justify left)
 		)
 	)
@@
 	(hierarchical_label "CLK8_FX_P"
 		(shape input)
-		(at 270.51 110.49 180)
-		(effects
-			(font
-				(size 1.27 1.27)
-			)
-			(justify right)
+		(at 223.52 72.39 0)
+		(effects
+			(font
+				(size 1.27 1.27)
+			)
+			(justify left)
 		)
 	)
@@
 	(hierarchical_label "CLK6_FX_N"
 		(shape input)
-		(at 270.51 92.71 180)
-		(effects
-			(font
-				(size 1.27 1.27)
-			)
-			(justify right)
+		(at 223.52 54.61 0)
+		(effects
+			(font
+				(size 1.27 1.27)
+			)
+			(justify left)
 		)
 	)
@@
 	(hierarchical_label "CLK2_FX_P"
 		(shape input)
-		(at 270.51 64.77 180)
+		(at 163.83 64.77 180)
 		(effects
 			(font
@@
 		)
 	)
-	(hierarchical_label "CLK5_FX_P"
-		(shape input)
-		(at 270.51 87.63 180)
-		(effects
-			(font
-				(size 1.27 1.27)
-			)
-			(justify right)
-		)
-	)
 	(hierarchical_label "CLK7_FX_N"
 		(shape input)
-		(at 270.51 100.33 180)
-		(effects
-			(font
-				(size 1.27 1.27)
-			)
-			(justify right)
+		(at 223.52 64.77 0)
+		(effects
+			(font
+				(size 1.27 1.27)
+			)
+			(justify left)
 		)
 	)
@@
 	(hierarchical_label "CLK6_FX_P"
 		(shape input)
-		(at 270.51 95.25 180)
-		(effects
-			(font
-				(size 1.27 1.27)
-			)
-			(justify right)
+		(at 223.52 52.07 0)
+		(effects
+			(font
+				(size 1.27 1.27)
+			)
+			(justify left)
 		)
 	)
@@
 	(hierarchical_label "CLK1_FX_N"
 		(shape input)
-		(at 270.51 54.61 180)
+		(at 163.83 52.07 180)
 		(effects
 			(font
@@
 	(hierarchical_label "CLK3_FX_N"
 		(shape input)
-		(at 270.51 69.85 180)
+		(at 163.83 77.47 180)
 		(effects
 			(font
@@
 		)
 	)
+	(hierarchical_label "CLK4_FX_N"
+		(shape input)
+		(at 163.83 92.71 180)
+		(effects
+			(font
+				(size 1.27 1.27)
+			)
+			(justify right)
+		)
+	)
 	(hierarchical_label "CLK7_FX_P"
 		(shape input)
-		(at 270.51 102.87 180)
-		(effects
-			(font
-				(size 1.27 1.27)
-			)
-			(justify right)
+		(at 223.52 62.23 0)
+		(effects
+			(font
+				(size 1.27 1.27)
+			)
+			(justify left)
 		)
 	)
@@
 		)
 	)
-	(hierarchical_label "CLK4_FX_P"
-		(shape input)
-		(at 270.51 80.01 180)
-		(effects
-			(font
-				(size 1.27 1.27)
-			)
-			(justify right)
-		)
-	)
 	(hierarchical_label "LCD_B7"
 		(shape output)
@@
 	(hierarchical_label "CLK3_FX_P"
 		(shape input)
-		(at 270.51 72.39 180)
+		(at 163.83 80.01 180)
 		(effects
 			(font
@@
 	(hierarchical_label "CLK1_FX_P"
 		(shape input)
-		(at 270.51 57.15 180)
-		(effects
-			(font
+		(at 163.83 54.61 180)
+		(effects
+			(font

Commit message: sch update
Connections:
- net IO0: now reaches M1.J2_41 (41)
- net IO1: now reaches M1.J2_43 (43)
- net IO2: now reaches M1.J2_45 (45)
- net IO3: now reaches M1.J2_47 (47)
- net IO4: now reaches M1.J2_49 (49)
- net IO5: now reaches M1.J2_51 (51)
- net IO6: now reaches M1.J2_53 (53)
- net IO7: now reaches M1.J2_57 (57)
- net IO8: now reaches M1.J2_59 (59)
- net IO9: now reaches M1.J2_61 (61)
- no-connect marks 4 -> 6
Changed lines of the file:
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@@
+	)
+	(no_connect
+		(at 77.47 41.91)
 	)
 	(no_connect
@@
 		(at 77.47 146.05)
 	)
+	(no_connect
+		(at 105.41 41.91)
+	)
 	(polyline
 		(pts
@@
 		(shape output)
 		(at 119.38 67.31 0)
+		(effects
+			(font
+				(size 1.27 1.27)
+			)
+			(justify left)
+		)
+	)
+	(hierarchical_label "IO4"
+		(shape bidirectional)
+		(at 223.52 92.71 0)
 		(effects
 			(font
@@
 		)
 	)
+	(hierarchical_label "IO5"
+		(shape bidirectional)
+		(at 223.52 95.25 0)
+		(effects
+			(font
+				(size 1.27 1.27)
+			)
+			(justify left)
+		)
+	)
 	(hierarchical_label "PL_LED0"
 		(shape output)
@@
 		)
 	)
+	(hierarchical_label "IO2"
+		(shape bidirectional)
+		(at 223.52 87.63 0)
+		(effects
+			(font
+				(size 1.27 1.27)
+			)
+			(justify left)
+		)
+	)
 	(hierarchical_label "LCD_R2"
 		(shape output)
@@
 		)
 	)
+	(hierarchical_label "IO1"
+		(shape bidirectional)
+		(at 223.52 85.09 0)
+		(effects
+			(font
+				(size 1.27 1.27)
+			)
+			(justify left)
+		)
+	)
 	(hierarchical_label "LCD_CLK"
 		(shape output)
@@
 		(shape output)
 		(at 119.38 72.39 0)
+		(effects
+			(font
+				(size 1.27 1.27)
+			)
+			(justify left)
+		)
+	)
+	(hierarchical_label "IO8"
+		(shape bidirectional)
+		(at 223.52 105.41 0)
 		(effects
 			(font
@@
 		)
 	)
+	(hierarchical_label "IO3"
+		(shape bidirectional)
+		(at 223.52 90.17 0)
+		(effects
+			(font
+				(size 1.27 1.27)
+			)
+			(justify left)
+		)
+	)
 	(hierarchical_label "PS_RXD"
 		(shape input)
@@
 		)
 	)
+	(hierarchical_label "IO0"
+		(shape bidirectional)
+		(at 223.52 82.55 0)
+		(effects
+			(font
+				(size 1.27 1.27)
+			)
+			(justify left)
+		)
+	)
+	(hierarchical_label "IO7"
+		(shape bidirectional)
+		(at 223.52 102.87 0)
+		(effects
+			(font
+				(size 1.27 1.27)
+			)
+			(justify left)
+		)
+	)
 	(hierarchical_label "XADC_VP"
 		(shape input)
@@
 		(shape output)
 		(at 119.38 90.17 0)
+		(effects
+			(font
+				(size 1.27 1.27)
+			)
+			(justify left)
+		)
+	)
+	(hierarchical_label "IO9"
+		(shape bidirectional)
+		(at 223.52 107.95 0)
 		(effects
 			(font
@@
 		)
 	)
+	(hierarchical_label "IO6"
+		(shape bidirectional)
+		(at 223.52 97.79 0)
+		(effects
+			(font
+				(size 1.27 1.27)
+			)
+			(justify left)
+		)
+	)
