File: hardware/schematic/v1.0/CORE/ZynqCore.kicad_sch (KiCad schematic)
At the start: 1 part, among them M1 ZYNQ7010&7020

Commit message: sch and pcb update
Connections:
- no-connect marks 27 -> 29
Changed lines of the file:
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@@
+	)
+	(no_connect
+		(at 62.23 54.61)
 	)
 	(no_connect
@@
 	)
 	(no_connect
+		(at 62.23 57.15)
+	)
+	(no_connect
