File: hardware/schematic/v1.0/CORE/Power.kicad_sch (KiCad schematic)
At the start: 11 parts, among them U2 TPS78633, U5 AMS1117-1.8

Commit message: sch update
Parts:
- added C11, C6: 100nF, Capacitor_SMD:C_0402_1005Metric, symbol Device:C
- added C12, C7: 10uF, Capacitor_SMD:C_0603_1608Metric, symbol Device:C
- added J10: USB_C_Receptacle_USB2.0_16P, Connector_USB:USB_C_Receptacle_Palconn_UTC16-G, symbol Connector:USB_C_Receptacle_USB2.0_16P
- added R36, R37: 5.1K, Resistor_SMD:R_0402_1005Metric, symbol Device:R
Connections:
- net GND: now also C11.2, C12.2, C6.2, C7.2, J10.A1 (GND), J10.A12 (GND), J10.B1 (GND), J10.B12 (GND), J10.SH (SHIELD), R36.2, R37.1
- net +5V renamed +VBUS_5V
- net +VBUS_5V: now also C11.1, C12.1, C6.1, C7.1, J10.A4 (VBUS), J10.A9 (VBUS), J10.B4 (VBUS), J10.B9 (VBUS)
- new net: J10.A5 (CC1), R36.1
- new net: J10.B5 (CC2), R37.2
- new net USB_D+: J10.A6 (D+), J10.B6 (D+)
- new net USB_D-: J10.A7 (D-), J10.B7 (D-)
- no-connect marks 0 -> 2
Other:
- note added: "DC IN"
- note added: "LDO"
- note removed: "POWER"
- moved on the sheet: C10, C15, C16, C17, C18, C19, C8, C9, R40, U2, U5

Commit message: sch update
Connections:
- net USB_D+: no longer names the net of J10.A6 (D+)
- net USB_D+: no longer J10.B6 (D+)
- net USB_D-: no longer names the net of J10.A7 (D-)
- net USB_D-: no longer J10.B7 (D-)
- no-connect marks 2 -> 6
Changed lines of the file:
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@@
-	)
-	(junction
-		(at 107.95 116.84)
-		(diameter 0)
-		(color 0 0 0 0)
 	)
 	(junction
@@
 	)
 	(junction
-		(at 107.95 109.22)
-		(diameter 0)
-		(color 0 0 0 0)
-	)
-	(junction
 		(at 140.97 96.52)
 		(diameter 0)
@@
 	)
 	(no_connect
+		(at 107.95 109.22)
+	)
+	(no_connect
 		(at 107.95 124.46)
+	)
+	(no_connect
+		(at 107.95 111.76)
+	)
+	(no_connect
+		(at 107.95 116.84)
+	)
+	(no_connect
+		(at 107.95 114.3)
 	)
 	(no_connect
 		(at 107.95 127)
 	)
-	(wire
-		(pts
-			(xy 107.95 109.22) (xy 111.76 109.22)
-		)
-		(stroke
-			(width 0)
-			(type default)
-		)
-	)
 	(polyline
 		(pts
@@
 	(wire
 		(pts
-			(xy 107.95 116.84) (xy 111.76 116.84)
-		)
-		(stroke
-			(width 0)
-			(type default)
-		)
-	)
-	(wire
-		(pts
 			(xy 152.4 39.37) (xy 154.94 39.37)
 		)
@@
 	(wire
 		(pts
-			(xy 107.95 109.22) (xy 107.95 111.76)
-		)
-		(stroke
-			(width 0)
-			(type default)
-		)
-	)
-	(wire
-		(pts
 			(xy 92.71 134.62) (xy 92.71 135.89)
 		)
@@
 	(wire
 		(pts
-			(xy 107.95 114.3) (xy 107.95 116.84)
-		)
-		(stroke
-			(width 0)
-			(type default)
-		)
-	)
-	(wire
-		(pts
 			(xy 81.28 46.99) (xy 85.09 46.99)
 		)
@@
 			(width 0)
 			(type default)
-		)
-	)
-	(global_label "USB_D-"
-		(shape output)
-		(at 111.76 109.22 0)
-		(fields_autoplaced yes)
-		(effects
-			(font
-				(size 1.27 1.27)
-			)
-			(justify left)
-		)
-		(property "Intersheetrefs" "${INTERSHEET_REFS}"
-			(at 122.3652 109.22 0)
-			(hide yes)
-			(show_name no)
-			(do_not_autoplace no)
-			(effects
-				(font
-					(size 1.27 1.27)
-				)
-				(justify left)
-			)
-		)
-	)
-	(global_label "USB_D+"
-		(shape input)
-		(at 111.76 116.84 0)
-		(fields_autoplaced yes)
-		(effects
-			(font
-				(size 1.27 1.27)
-			)
-			(justify left)
-		)
-		(property "Intersheetrefs" "${INTERSHEET_REFS}"
-			(at 122.3652 116.84 0)
-			(hide yes)
-			(show_name no)
-			(do_not_autoplace no)
-			(effects
-				(font
-					(size 1.27 1.27)
-				)
-				(justify left)
-			)
 		)
 	)
@@
 		)
 		(property "Value" "+VBUS_5V"
-			(at 133.35 90.17 0)
-			(show_name no)
-			(do_not_autoplace no)
-			(effects
-				(font
-					(size 1.27 1.27)
-				)
-			)
-		)
+			(at 135.89 93.9799 0)
+			(show_name no)
+			(do_not_autoplace no)
+			(effects
+				(font
+					(size 1.27 1.27)
+				)
+				(justify right)
+			)
+		)

Commit message: sch update
Parts:
- added C26: 10uF, Capacitor_SMD:C_0603_1608Metric, symbol Device:C
- added C27: 100nF, Capacitor_SMD:C_0402_1005Metric, symbol Device:C
- added CN1: LAIL-PHC2_54-2P-01-XH-L, JLCImport:LAIL-PHC2_54-2P-01-XH-L, symbol JLCImport:LAIL-PHC2_54-2P-01-XH-L
- added D7: LED, LED_SMD:LED_0603_1608Metric, symbol Device:LED
- added F2: BSMD1206C-1300T, JLCImport:BSMD1206C-1300T, symbol JLCImport:BSMD1206C-1300T
- added R45: 1K, Resistor_SMD:R_0402_1005Metric, symbol Device:R
Connections:
- net GND: now also C26.2, C27.2, CN1.2, D7.1 (K)
- net +VBUS_5V renamed +5V_IN
- net +5V_IN: now also C26.1, C27.1, CN1.1, F2.1; no longer R40.2, U2.2 (IN)
- new net: D7.2 (A), R45.2
- new net +5V: F2.2, R40.2, R45.1, U2.2 (IN)
Other:
- note added: "5V"
- note added: "PHC IN"
- moved on the sheet: C10, C11, C12, C15, C16, C17, C18, C19, C6, C7, C8, C9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

Commit message: sch update
Parts:
- added D8, D9: SS34, Diode_SMD:D_SMA, symbol Diode:SS34
Connections:
- net +5V_IN: now also D9.2 (A); no longer C11.1, C12.1, C6.1, C7.1, F2.1, J10.A4 (VBUS), J10.A9 (VBUS), J10.B4 (VBUS), J10.B9 (VBUS)
- new net: D8.1 (K), D9.1 (K), F2.1
- new net +VBUS_5V: C11.1, C12.1, C6.1, C7.1, D8.2 (A), J10.A4 (VBUS), J10.A9 (VBUS), J10.B4 (VBUS), J10.B9 (VBUS)
Other:
- moved on the sheet: C26, C27
