File: hardware/schematic/v1.0/CORE_CAST/CORE_CAST.kicad_sch (KiCad schematic)
At the start: 0 parts

Commit message: update core_cast sch
Parts:
- added BOOT_CFG1: CSW-2P, Counter:CSW DIP-2P, symbol Counter:CSW-2P
- added C1, C11, C19, C2, C3, C5, C6: 100nF, Capacitor_SMD:C_0402_1005Metric, symbol Device:C
- added C10, C12, C15, C17, C7, C8: 10uF, Capacitor_SMD:C_0603_1608Metric, symbol Device:C
- added C16, C18: 100nF, Capacitor_SMD:C_0603_1608Metric, symbol Device:C
- added C4: 10uF, Capacitor_SMD:C_0402_1005Metric, symbol Device:C
- added C9: 10nF, Capacitor_SMD:C_0402_1005Metric, symbol Device:C
- added D1, D2: AZ1143-04F.R7G, Counter:DFN2510P10E, symbol Counter:AZ1045-04F.R7G
- added D3, D4, D5, D6: LED, LED_SMD:LED_0603_1608Metric, symbol Device:LED
- added GE_PS1: HR911131A, Counter:HR911131A, symbol Counter:HR911131A_C
- added J1, J11: Conn_01x06_Socket, Connector_PinHeader_2.54mm:PinHeader_1x06_P2.54mm_Vertical, symbol Connector:Conn_01x06_Socket
- added J10: USB_C_Receptacle_USB2.0_16P, Connector_USB:USB_C_Receptacle_Palconn_UTC16-G, symbol Connector:USB_C_Receptacle_USB2.0_16P
- added J12, J2, J3, J4, J5, J6, J7, J8, J9: Conn_Coaxial, Connector_Coaxial:SMA_Amphenol_132289_EdgeMount, symbol Connector:Conn_Coaxial
- added J13, J16: Conn_01x04_Socket, Connector_PinHeader_2.54mm:PinHeader_1x04_P2.54mm_Vertical, symbol Connector:Conn_01x04_Socket
- added J14: Conn_01x03_Socket, Connector_PinHeader_2.54mm:PinHeader_1x03_P2.54mm_Vertical, symbol Connector:Conn_01x03_Socket
- added J15: Conn_01x05_Socket, Connector_PinHeader_2.54mm:PinHeader_1x05_P2.54mm_Vertical, symbol Connector:Conn_01x05_Socket
- added JTAG1: JTAG, Counter:DC3_14P_2_7_DIP, symbol Counter:Header 7X2
- added M1: ZYNQ7010&7020, Counter:ZYNQ7010&7020_CB, symbol Counter:ZYNQ7010&7020
- added R1, R2, R3, R4: 33R, Resistor_SMD:R_0402_1005Metric, symbol Device:R
- added R10, R5, R6, R7, R8, R9: 499R, Resistor_SMD:R_0402_1005Metric, symbol Device:R
- added R11, R12: 20K, Resistor_SMD:R_0402_1005Metric, symbol Device:R
- added R13, R14, R18: 10K, Resistor_SMD:R_0402_1005Metric, symbol Device:R
- added R15, R19, R20, R21, R22, R23: 4.7K, Resistor_SMD:R_0402_1005Metric, symbol Device:R
- added R16: 330, Resistor_SMD:R_0402_1005Metric, symbol Device:R
- added R17, R38, R39, R40: 0, Resistor_SMD:R_0402_1005Metric, symbol Device:R
- added R36, R37: 5.1K, Resistor_SMD:R_0402_1005Metric, symbol Device:R
- added U1: TXS02612RTWR, Counter:QFN24_RTW, symbol Counter:TXS02612RTWR
- added U2: TPS78633, Package_TO_SOT_SMD:SOT-223-6, symbol Counter:TPS78633
- added U3: SD_Card, Counter:SIM-SMD_LX_XDFP-0090-012, symbol Counter:SD_Card
- added U5: AMS1117-1.8, Package_TO_SOT_SMD:SOT-223-3_TabPin2, symbol Regulator_Linear:AMS1117-1.8
- added U6: CH340E, Package_SO:MSOP-10_3x3mm_P0.5mm, symbol Interface_USB:CH340E
Connections:
- new net: R39.2, U6.9 (RXD)
- new net: D6.2 (A), R8.2
- new net: R23.2, U1.23 (DAT2B0), U3.1 (DAT2)
- new net: R22.2, U1.22 (DAT3B0), U3.2 (CD/DAT3/CS)
- new net: R21.2, U1.20 (CMDB0), U3.3 (CMD/SDI)
- new net: U1.19 (CLKB0), U3.5 (CLK/SLCK)
- new net: R20.2, U1.18 (DAT0B0), U3.7 (DAT0/SDO)
- new net: R19.2, U1.16 (DAT1B0), U3.8 (DAT1)
- new net: R16.2, U3.9 (CD/SW)
- new net: R15.1, U1.24 (SEL)
- new net: C9.2, U2.5 (NR/FB)
- new net: D3.2 (A), R5.2
- new net: JTAG1.4, R1.1
- new net: R38.1, U6.8 (TXD)
- new net: JTAG1.8, R3.1
- new net: JTAG1.6, R2.1
- new net: J10.A5 (CC1), R36.1
- new net: GE_PS1.11 (GA), R10.1
- new net: R16.1, R17.2, R18.2
- new net: D4.2 (A), R6.2
- new net: C8.2, R40.1, U2.1 (EN)
- new net: J10.B5 (CC2), R37.2
- new net: JTAG1.10, R4.1
- new net: BOOT_CFG1.3, R12.1, R14.1
- new net: BOOT_CFG1.4, R11.1, R13.1
- new net: GE_PS1.14 (YA), R9.2
- new net: D1.10 (NC), GE_PS1.1 (TX1+)
- new net: D2.6 (NC), GE_PS1.10 (TX4-)
- new net: D1.9 (NC), GE_PS1.2 (TX1-)
- new net: D1.7 (NC), GE_PS1.3 (TX2+)
- new net: D1.6 (NC), GE_PS1.4 (TX2-)
- new net: C1.1, GE_PS1.5 (CT1), GE_PS1.6 (CT2)
- new net: D2.10 (NC), GE_PS1.7 (TX3+)
- new net: D2.9 (NC), GE_PS1.8 (TX3-)
- new net: D2.7 (NC), GE_PS1.9 (TX4+)
- new net: D5.2 (A), R7.2
- new net +1.8V: C17.1, C18.1, C3.2, U1.5 (VCCA), U5.2 (VO)
- new net +3.3V: C10.2, C15.1, C16.1, C19.2, C2.2, C4.1, C5.1, J1.3 (Pin_3), J1.4 (Pin_4), J11.3 (Pin_3), J11.4 (Pin_4), JTAG1.2, R10.2, R13.2, R14.2, R18.1, R19.1, R20.1, R21.1, R22.1, R23.1, R9.1, U1.17 (VCCB1), U1.21 (VCCB0), U2.4 (OUT), U3.4 (VDD), U5.3 (VI), U6.10 (V3), U6.7 (VCC)
- new net +5V: C11.1, C12.1, C6.1, C7.1, J1.1 (Pin_1), J1.2 (Pin_2), J10.A4 (VBUS), J10.A9 (VBUS), J10.B4 (VBUS), J10.B9 (VBUS), J11.1 (Pin_1), J11.2 (Pin_2), M1.J1_1 (1), M1.J1_2 (2), M1.J1_3 (3), M1.J1_4 (4), M1.J1_5 (5), M1.J1_6 (6), M1.J1_7 (7), M1.J1_8 (8), R40.2, U2.2 (IN)
- new net BOOT_MODE0: M1.J2_81 (81), R11.2
- new net BOOT_MODE1: M1.J2_79 (79), R12.2
- new net CLK1_FS_N: J9.1 (In), M1.J1_48 (48)
- new net CLK1_FS_P: J8.1 (In), M1.J1_50 (50)
- new net CLK1_FX_N: J7.1 (In), M1.J2_38 (38)
- new net CLK1_FX_P: J6.1 (In), M1.J2_40 (40)
- new net CLK_10M: J12.1 (In)
- new net CLK_FS_N: J5.1 (In), M1.J1_18 (18)
- new net CLK_FS_P: J4.1 (In), M1.J1_16 (16)
- new net CLK_FX_N: J3.1 (In), M1.J2_26 (26)
- new net CLK_FX_P: J2.1 (In), M1.J2_28 (28)
- new net FPGA_TCK: M1.J2_99 (99), R2.2
- new net FPGA_TDI: M1.J2_98 (98), R4.2
- new net FPGA_TDO: M1.J2_97 (97), R3.2
- new net FPGA_TMS: M1.J2_100 (100), R1.2
- new net GND: BOOT_CFG1.1, BOOT_CFG1.2, C1.2, C10.1, C11.2, C12.2, C15.2, C16.2, C17.2, C18.2, C19.1, C2.1, C3.1, C4.2, C5.2, C6.2, C7.2, C8.1, C9.1, D1.3 (GND), D1.8 (GND), D2.3 (GND), D2.8 (GND), D3.1 (K), D4.1 (K), D5.1 (K), D6.1 (K), GE_PS1.15 (GND), GE_PS1.16 (GND), J1.5 (Pin_5), J1.6 (Pin_6), J10.A1 (GND), J10.A12 (GND), J10.B1 (GND), J10.B12 (GND), J10.SH (SHIELD), J11.5 (Pin_5), J11.6 (Pin_6), J12.2 (Ext), J14.3 (Pin_3), J15.5 (Pin_5), J2.2 (Ext), J3.2 (Ext), J4.2 (Ext), J5.2 (Ext), J6.2 (Ext), J7.2 (Ext), J8.2 (Ext), J9.2 (Ext), JTAG1.1, JTAG1.11, JTAG1.13, JTAG1.3, JTAG1.5, JTAG1.7, JTAG1.9, M1.J1_100 (100), M1.J1_19 (19), M1.J1_34 (34), M1.J1_41 (41), M1.J1_52 (52), M1.J1_59 (59), M1.J1_70 (70), M1.J1_93 (93), M1.J1_94 (94), M1.J1_95 (95), M1.J1_96 (96), M1.J1_97 (97), M1.J1_98 (98), M1.J1_99 (99), M1.J2_11 (11), M1.J2_12 (12), M1.J2_62 (62), M1.J2_63 (63), M1.J2_76 (76), M1.J2_77 (77), R15.2, R36.2, R37.1, U1.11 (GND2), U1.2 (GND1), U1.25 (EPAD), U2.3 (GND), U2.6 (TAB), U3.10 (GND), U3.11 (GND), U3.12 (GND), U3.13 (GND), U3.6 (VSS), U5.1 (GND), U6.3 (GND)
- new net I2C_SCL: J14.2 (Pin_2), M1.J2_65 (65)
- new net I2C_SDA: J14.1 (Pin_1), M1.J2_70 (70)
- new net IO0: J13.1 (Pin_1), M1.J1_43 (43)
- new net IO1: J13.2 (Pin_2), M1.J1_45 (45)
- new net IO2: J13.3 (Pin_3), M1.J1_47 (47)
- new net IO3: J13.4 (Pin_4), M1.J1_49 (49)
- new net IO4: J16.1 (Pin_1), M1.J1_51 (51)
- new net IO5: J16.2 (Pin_2), M1.J1_53 (53)
- new net IO6: J16.3 (Pin_3), M1.J1_55 (55)
- new net IO7: J16.4 (Pin_4), M1.J1_57 (57)
- new net PHY1_AD0/LED0: GE_PS1.12 (GC), M1.J2_1 (1)
- new net PHY1_AD1/LED1: GE_PS1.13 (YC), M1.J2_2 (2)
- new net PHY1_MDI0_N: D1.2 (Line-2), M1.J2_5 (5)
- new net PHY1_MDI0_P: D1.1 (Line-1), M1.J2_3 (3)
- new net PHY1_MDI1_N: D1.5 (Line-4), M1.J2_9 (9)
- new net PHY1_MDI1_P: D1.4 (Line-3), M1.J2_7 (7)
- new net PHY1_MDI2_N: D2.2 (Line-2), M1.J2_6 (6)
- new net PHY1_MDI2_P: D2.1 (Line-1), M1.J2_4 (4)
- new net PHY1_MDI3_N: D2.5 (Line-4), M1.J2_10 (10)
- new net PHY1_MDI3_P: D2.4 (Line-3), M1.J2_8 (8)
- new net PL_LED0: M1.J2_44 (44), R5.1
- new net PL_LED1: M1.J2_55 (55), R6.1
- new net PS_LED0: M1.J2_92 (92), R7.1
- new net PS_LED1: M1.J2_95 (95), R8.1
- new net RXD: M1.J2_89 (89), R38.2
- new net SD_CD: M1.J2_96 (96), R17.1
- new net SD_CLK: M1.J2_80 (80), U1.9 (CLKA)
- new net SD_CMD: M1.J2_78 (78), U1.4 (CMDA)
- new net SD_D0: M1.J2_82 (82), U1.6 (DAT0A)
- new net SD_D1: M1.J2_84 (84), U1.7 (DAT1A)
- new net SD_D2: M1.J2_86 (86), U1.1 (DAT2A)
- new net SD_D3: M1.J2_88 (88), U1.3 (DAT3A)
- new net SPI1_MISO: J15.2 (Pin_2), M1.J2_94 (94)
- new net SPI1_MOSI: J15.1 (Pin_1), M1.J2_91 (91)
- new net SPI1_SCLK: J15.3 (Pin_3), M1.J2_90 (90)
- new net SPI1_SS0: J15.4 (Pin_4), M1.J2_93 (93)
- new net TXD: M1.J2_87 (87), R39.1
- new net USB_D+: J10.A6 (D+), J10.B6 (D+), U6.1 (UD+)
- new net USB_D-: J10.A7 (D-), J10.B7 (D-), U6.2 (UD-)
- new net XADC_VN: M1.J2_85 (85)
- new net XADC_VP: M1.J2_83 (83)
- no-connect marks 0 -> 132
Other:
- note added: "B35_L2_N_A20"
- note added: "B35_L2_P_B19"
- note added: "ETHERNET(PS)"
- note added: "JTAG"
- note added: "MIO 4"
- note added: "MIO 5"
- note added: "MRCC B34_L13_N P19"
- note added: "MRCC B34_L13_P N18"
- note added: "MRCC B35_L12_N K18"
- note added: "MRCC B35_L12_P K17"
- note added: "MRCC B35_L13_N H17"
- note added: "MRCC B35_L13_P H16"
- note added: "POWER"
- note added: "PS/PL LED"
- note added: "PS_MIO10"
- note added: "PS_MIO11"
- note added: "PS_MIO12"
- note added: "PS_MIO13"
- note added: "PS_MIO30"
- note added: "PS_MIO31"
- note added: "PS_MIO40"
- note added: "PS_MIO41"
- note added: "PS_MIO42"
- note added: "PS_MIO43"
- note added: "PS_MIO44"
- note added: "PS_MIO45"
- note added: "PS_MIO7"
- note added: "PS_MIO8"
- note added: "PS_MIO9"
- note added: "SD_CARD"
- note added: "SIGNAL"
- note added: "SOCKET"
- note added: "SRCC B34_L11_N U15"
- note added: "SRCC B34_L11_P U14"
- note added: "SRCC B34_L14_N P20"
- note added: "SRCC B34_L14_P N20"
- note added: "SRCC B35_L11_N L17"
- note added: "SRCC B35_L11_P L16"
- note added: "SRCC B35_L14_N H18"
- note added: "SRCC B35_L14_P J18"

Commit message: sch updaate
Parts:
- added J17, J18, J19, J20, J21, J22, J23, J24: Conn_Coaxial, Connector_Coaxial:SMA_Amphenol_132289_EdgeMount, symbol Connector:Conn_Coaxial
- added U4: *, Counter:STAMP_HOLES_154P_C, symbol Counter:154PIN_Stamp_holes_0
Connections:
- net BOOT_MODE0: now also U4.127
- net BOOT_MODE1: now also U4.126
- net CLK1_FS_N: now also J22.1 (In), U4.2
- net CLK1_FS_P: now also J21.1 (In), U4.1
- net CLK1_FX_N: now also J20.1 (In), U4.89
- net CLK1_FX_P: now also J19.1 (In), U4.90
- net CLK_FS_N: now also J24.1 (In), U4.44
- net CLK_FS_P: now also J23.1 (In), U4.45
- net CLK_FX_N: now also J18.1 (In), U4.84
- net CLK_FX_P: now also J17.1 (In), U4.85
- net FPGA_TCK: now also U4.146
- net FPGA_TDI: now also U4.144
- net FPGA_TDO: now also U4.145
- net FPGA_TMS: now also U4.143
- net GND: now also J17.2 (Ext), J18.2 (Ext), J19.2 (Ext), J20.2 (Ext), J21.2 (Ext), J22.2 (Ext), J23.2 (Ext), J24.2 (Ext), U4.106, U4.133, U4.136, U4.19, U4.29, U4.46, U4.69, U4.86, U4.9, U4.95
- net PHY1_AD0/LED0: now also U4.92
- net PHY1_AD1/LED1: now also U4.91
- net PHY1_MDI0_N: now also U4.98
- net PHY1_MDI0_P: now also U4.97
- net PHY1_MDI1_N: now also U4.100
- net PHY1_MDI1_P: now also U4.99
- net PHY1_MDI2_N: now also U4.102
- net PHY1_MDI2_P: now also U4.101
- net PHY1_MDI3_N: now also U4.104
- net PHY1_MDI3_P: now also U4.103
- net PS_LED0: now also U4.121
- net PS_LED1: now also U4.125
- net RXD: now also U4.120
- net SD_CLK: now also U4.138
- net SD_CMD: now also U4.128
- net SD_D0: now also U4.131
- net SD_D1: now also U4.132
- net SD_D2: now also U4.129
- net SD_D3: now also U4.137
- net SPI1_MISO: now also U4.123
- net SPI1_MOSI: now also U4.122
- net SPI1_SCLK: now also U4.118
- net SPI1_SS0: now also U4.124
- net TXD: now also U4.119
- new net BTC_3V3: U4.134, U4.135
- new net VCCIO_B34: U4.18
- new net VCCIO_B35: U4.96
- no-connect marks 132 -> 134
Other:
- note added: "B34_IO25"
- note added: "B34_L10_N"
- note added: "B34_L10_P"
- note added: "B34_L15_N"
- note added: "B34_L15_P"
- note added: "B34_L16_N"
- note added: "B34_L16_P"
- note added: "B34_L17_N"
- note added: "B34_L17_P"
- note added: "B34_L18_N"
- note added: "B34_L18_P"
- note added: "B34_L19_N"
- note added: "B34_L19_P"
- note added: "B34_L1_N"
- note added: "B34_L1_P"
- note added: "B34_L20_N"
- note added: "B34_L20_P"
- note added: "B34_L21_N"
- note added: "B34_L21_P"
- note added: "B34_L22_N"
- note added: "B34_L22_P"
- note added: "B34_L23_N"
- note added: "B34_L23_P"
- note added: "B34_L24_N"
- note added: "B34_L24_P"
- note added: "B34_L2_N"
- note added: "B34_L2_P"
- note added: "B34_L3_N"
- note added: "B34_L3_P"
- note added: "B34_L4_N"
- note added: "B34_L4_P"
- note added: "B34_L5_N"
- note added: "B34_L5_P"
- note added: "B34_L6_N"
- note added: "B34_L6_P"
- note added: "B34_L7_N"
- note added: "B34_L7_P"
- note added: "B34_L8_N"
- note added: "B34_L8_P"
- note added: "B34_L9_N"
- note added: "B34_L9_P"
- note added: "B34_LO0"
- note added: "B35_IO25"
- note added: "B35_L10_N"
- note added: "B35_L10_P"
- note added: "B35_L11_N"
- note added: "B35_L11_P"
- note added: "B35_L15_N"
- note added: "B35_L15_P"
- note added: "B35_L16_N"
- note added: "B35_L16_P"
- note added: "B35_L17_N"
- note added: "B35_L17_P"
- note added: "B35_L18_N"
- note added: "B35_L18_P"
- note added: "B35_L19_N"
- note added: "B35_L19_P"
- note added: "B35_L1_N"
- note added: "B35_L1_P"
- note added: "B35_L20_N"
- note added: "B35_L20_P"
- note added: "B35_L21_N"
- note added: "B35_L21_P"
- note added: "B35_L22_N"
- note added: "B35_L22_P"
- note added: "B35_L23_N"
- note added: "B35_L23_P"
- note added: "B35_L24_N"
- note added: "B35_L24_P"
- note added: "B35_L2_N"
- note added: "B35_L2_P"
- note added: "B35_L3_N"
- note added: "B35_L3_P"
- note added: "B35_L4_N"
- note added: "B35_L4_P"
- note added: "B35_L5_N"
- note added: "B35_L5_P"
- note added: "B35_L6_N"
- note added: "B35_L6_P"
- note added: "B35_L7_N"
- note added: "B35_L7_P"
- note added: "B35_L8_N"
- note added: "B35_L8_P"
- note added: "B35_L9_N"
- note added: "B35_L9_P"
- note added: "B35_LO0"
- note added: "BO_VN"
- note added: "BO_VP"
- note added: "CLK1_FS"
- note added: "CLK_FS"
- note added: "CLK_FX"
- note added: "FPGA_TCK"
- note added: "FPGA_TDI"
- note added: "FPGA_TDO"
- note added: "FPGA_TMS"
- note added: "OTG_D_N"
- note added: "OTG_D_P"
- note added: "OTG_ID"
- note added: "OTG_RESETN"
- note added: "PHY_AD0/LED0"
- note added: "PHY_AD1/LED1"
- note added: "PHY_MDI0_N"
- note added: "PHY_MDI0_P"
- note added: "PHY_MDI1_N"
- note added: "PHY_MDI1_P"
- note added: "PHY_MDI2_N"
- note added: "PHY_MDI2_P"
- note added: "PHY_MDI3_N"
- note added: "PHY_MDI3_P"
- note added: "PS_MIO14"
- note added: "PS_MIO15"
- note added: "PS_MIO4"
- note added: "PS_MIO5"
- note added: "PS_PRO_B"
- note added: "PW_GOOD"
- note added: "USB_VBUS"
- note added: "VUSB_V_EN"
- moved on the sheet: BOOT_CFG1, C1, C10, C11, C12, C15, C16, C17, C18, C19, C2, C3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

Commit message: sch update
Parts:
- added RGB TFTLCD1: RGBLCD, AD:FPC-TOP40, symbol Counter:FPC-40
Connections:
- net +3.3V: now also RGB TFTLCD1.4
- net GND: now also RGB TFTLCD1.29, RGB TFTLCD1.3, RGB TFTLCD1.36, RGB TFTLCD1.A, RGB TFTLCD1.B
- net PL_LED0: now also U4.94
- net PL_LED1: now also U4.113
- net G4: now reaches U4.10
- net G4: now also RGB TFTLCD1.17
- net G5: now reaches U4.11
- net G5: now also RGB TFTLCD1.18
- net G6: now reaches U4.12
- net G6: now also RGB TFTLCD1.19
- net G7: now reaches U4.13
- net G7: now also RGB TFTLCD1.20
- net B0: now reaches U4.14
- net B0: now also RGB TFTLCD1.21
- net R0: now reaches U4.147
- net R0: now also RGB TFTLCD1.5
- net R1: now reaches U4.148
- net R1: now also RGB TFTLCD1.6
- net R2: now reaches U4.149
- net R2: now also RGB TFTLCD1.7
- net B1: now reaches U4.15
- net B1: now also RGB TFTLCD1.22
- net R3: now reaches U4.150
- net R3: now also RGB TFTLCD1.8
- net R4: now reaches U4.151
- net R4: now also RGB TFTLCD1.9
- net R5: now reaches U4.152
- net R5: now also RGB TFTLCD1.10
- net R6: now reaches U4.153
- net R6: now also RGB TFTLCD1.11
- net B2: now reaches U4.16
- net B2: now also RGB TFTLCD1.23
- net B3: now reaches U4.17
- net B3: now also RGB TFTLCD1.24
- net B4: now reaches U4.20
- net B4: now also RGB TFTLCD1.25
- net B5: now reaches U4.21
- net B5: now also RGB TFTLCD1.26
- net B6: now reaches U4.22
- net B6: now also RGB TFTLCD1.27
- net B7: now reaches U4.23
- net B7: now also RGB TFTLCD1.28
- net DE: now reaches U4.33
- net DE: now also RGB TFTLCD1.34
- net CLK: now reaches U4.34
- net CLK: now also RGB TFTLCD1.30
- net DISP: now reaches U4.35
- net DISP: now also RGB TFTLCD1.31
- net HSYNC: now reaches U4.36
- net HSYNC: now also RGB TFTLCD1.32
- net VSYNC: now reaches U4.37
- net VSYNC: now also RGB TFTLCD1.33
- net G0: now reaches U4.5
- net G0: now also RGB TFTLCD1.13
- net G1: now reaches U4.6
- net G1: now also RGB TFTLCD1.14
- net G2: now reaches U4.7
- net G2: now also RGB TFTLCD1.15
- net G3: now reaches U4.8
- net G3: now also RGB TFTLCD1.16
- new net R7: RGB TFTLCD1.12
- no-connect marks 134 -> 139
Other:
- note added: "RGB888"
- moved on the sheet: J21, J22

Commit message: sch update
Parts:
- added J25: HDMI_A, Connector_Video:HDMI_A_Molex_208658-1001_Horizontal, symbol Connector:HDMI_A
- added U7: FPC-6P, symbol Counter:FPC-6P
Connections:
- net +3.3V: now also U7.2
- net GND: now also U7.3, U7.7 (SH), U7.8 (SH)
- new net CTP_INT: U7.4
- new net CTP_RST: U7.1
- new net CTP_SCL: U7.6
- new net CTP_SDA: U7.5
Other:
- moved on the sheet: C2, C3, C4, C5, D3, D4, D5, D6, R15, R16, R17, R18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

Commit message: sch update
Connections:
- net B0: now also U4.12; no longer U4.14
- net B1: now also U4.13; no longer U4.15
- net B2: now also U4.14; no longer U4.16
- net B3: now also U4.15; no longer U4.17
- net B4: now also U4.16; no longer U4.20
- net B5: now also U4.17; no longer U4.21
- net B6: now also U4.20; no longer U4.22
- net B7: now also U4.21; no longer U4.23
- net CTP_INT: now also U4.24
- net CTP_RST: now also U4.25
- net CTP_SCL: now also U4.22
- net CTP_SDA: now also U4.23
- net G0: now also U4.3; no longer U4.5
- net G1: now also U4.4; no longer U4.6
- net G2: now also U4.5; no longer U4.7
- net G3: now also U4.6; no longer U4.8
- net G4: now also U4.7; no longer U4.10
- net G5: now also U4.8; no longer U4.11
- net G6: now also U4.10; no longer U4.12
- net G7: now also U4.11; no longer U4.13

Commit message: sch upate
Parts:
- added J26: Conn_01x04_Socket, Connector_PinHeader_2.54mm:PinHeader_1x04_P2.54mm_Vertical, symbol Connector:Conn_01x04_Socket
- added R41, R42: 49.9, Resistor_SMD:R_0402_1005Metric, symbol Device:R
Connections:
- net +3.3V: now also J26.1 (Pin_1)
- net GND: now also J26.4 (Pin_4)
- net XADC_VN: now also U4.141, R42.1
- net XADC_VP: now also U4.140, R41.2
- new net: J26.2 (Pin_2), R41.1
- new net: J26.3 (Pin_3), R42.2
Other:
- note added: "BO_VN L10"
- note added: "BO_VP K9"
- note added: "XADC"
- note removed: "BO_VN"
- note removed: "BO_VP"
- moved on the sheet: C10, C11, C12, C15, C16, C17, C18, C19, C6, C7, C8, C9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

Commit message: sch update
Parts:
- added C13: 1nF, Capacitor_SMD:C_0402_1005Metric, symbol Device:C
Connections:
- net B0: now also U4.8; no longer U4.12
- net B1: now also U4.7; no longer U4.13
- net B2: now also U4.6; no longer U4.14
- net B3: now also U4.5; no longer U4.15
- net B4: now also U4.4; no longer U4.16
- net B5: now also U4.3; no longer U4.17
- net B6: now also U4.154; no longer U4.20
- net B7: now also U4.153; no longer U4.21
- net CLK: now also U4.152; no longer U4.34
- net CTP_INT: now also U4.40; no longer U4.24
- net CTP_RST: now also U4.41; no longer U4.25
- net CTP_SCL: now also U4.38; no longer U4.22
- net CTP_SDA: now also U4.39; no longer U4.23
- net DE: now also U4.148; no longer U4.33
- net DISP: now also U4.151; no longer U4.35
- net G0: now also U4.17; no longer U4.3
- net G1: now also U4.16; no longer U4.4
- net G2: now also U4.15; no longer U4.5
- net G3: now also U4.14; no longer U4.6
- net G4: now also U4.13; no longer U4.7
- net G5: now also U4.12; no longer U4.8
- net G6: now also U4.11; no longer U4.10
- net G7: now also U4.10; no longer U4.11
- net HSYNC: now also U4.150; no longer U4.36
- net I2C_SCL: no longer J14.2 (Pin_2)
- net I2C_SDA: no longer J14.1 (Pin_1)
- net R0: now also U4.35; no longer U4.147
- net R1: now also U4.34; no longer U4.148
- net R2: now also U4.25; no longer U4.149
- net R3: now also U4.24; no longer U4.150
- net R4: now also U4.23; no longer U4.151
- net R5: now also U4.22; no longer U4.152
- net R6: now also U4.21; no longer U4.153
- net R7: now also U4.20
- net SPI1_MISO: no longer J15.2 (Pin_2), U4.123
- net SPI1_MOSI: no longer J15.1 (Pin_1), U4.122
- net SPI1_SCLK: no longer J15.3 (Pin_3), U4.118
- net SPI1_SS0: no longer J15.4 (Pin_4), U4.124
- net VSYNC: now also U4.149; no longer U4.37
- net at J26.2 (Pin_2), R41.1: now also C13.1
- net at J26.3 (Pin_3), R42.2: now also C13.2
- new net PS_I2C_SCL: J14.2 (Pin_2)
- new net PS_I2C_SDA: J14.1 (Pin_1)
- new net PS_SPI1_MISO: J15.2 (Pin_2), U4.123
- new net PS_SPI1_MOSI: J15.1 (Pin_1), U4.122
- new net PS_SPI1_SCLK: J15.3 (Pin_3), U4.118
- new net PS_SPI1_SS0: J15.4 (Pin_4), U4.124
Other:
- moved on the sheet: D3, D4, D5, D6, J1, J14, J26, R41, R42, R5, R6, R7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
