File: hardware/schematic/v1.0/CORE_Rev1.0/Display.kicad_sch (KiCad schematic)
At the start: 7 parts, among them Q1 Si2302CDS-T1-GE3, U7 FPC-6P

Commit message: sch update
Parts:
- removed RGB TFTLCD1: RGBLCD, AD:FPC-TOP40, symbol Counter:FPC-40
- removed U7: FPC-6P, symbol Counter:FPC-6P
- added RGB TFTLCD1: RGBLCD, CORE:LAIL-FPC-CDX01-40P0_5-GW, symbol CORE:FPC-40
- added U7: FPC-6P, CORE:FPC-05F-6PH20, symbol CORE:FPC-6P
Connections:
- net +3.3V: now also RGB TFTLCD1.1, RGB TFTLCD1.4, U7.2
- net CTP_INT: now also U7.4
- net CTP_RST: now also U7.1
- net CTP_SCL: now also U7.6
- net CTP_SDA: now also U7.5
- net GND: now also RGB TFTLCD1.29, RGB TFTLCD1.3, RGB TFTLCD1.36, RGB TFTLCD1.A, RGB TFTLCD1.B, U7.3, U7.7 (SH), U7.8 (SH)
- net LCD_B0: now also RGB TFTLCD1.21
- net LCD_B1: now also RGB TFTLCD1.22
- net LCD_B2: now also RGB TFTLCD1.23
- net LCD_B3: now also RGB TFTLCD1.24
- net LCD_B4: now also RGB TFTLCD1.25
- net LCD_B5: now also RGB TFTLCD1.26
- net LCD_B6: now also RGB TFTLCD1.27
- net LCD_B7: now also RGB TFTLCD1.28
- net LCD_CLK: now also RGB TFTLCD1.30
- net LCD_DE: now also RGB TFTLCD1.34
- net LCD_DISP: now also RGB TFTLCD1.31
- net LCD_G0: now also RGB TFTLCD1.13
- net LCD_G1: now also RGB TFTLCD1.14
- net LCD_G2: now also RGB TFTLCD1.15
- net LCD_G3: now also RGB TFTLCD1.16
- net LCD_G4: now also RGB TFTLCD1.17
- net LCD_G5: now also RGB TFTLCD1.18
- net LCD_G6: now also RGB TFTLCD1.19
- net LCD_G7: now also RGB TFTLCD1.20
- net LCD_HSYNC: now also RGB TFTLCD1.32
- net LCD_R0: now also RGB TFTLCD1.5
- net LCD_R1: now also RGB TFTLCD1.6
- net LCD_R2: now also RGB TFTLCD1.7
- net LCD_R3: now also RGB TFTLCD1.8
- net LCD_R4: now also RGB TFTLCD1.9
- net LCD_R5: now also RGB TFTLCD1.10
- net LCD_R6: now also RGB TFTLCD1.11
- net LCD_R7: now also RGB TFTLCD1.12
- net LCD_VSYNC: now also RGB TFTLCD1.33
- net LEDK: now also RGB TFTLCD1.2

Commit message: sch update
Parts:
- removed U7: FPC-6P, CORE:FPC-05F-6PH20, symbol CORE:FPC-6P
- added FPC1: FPC-05F-6PH20, CORE:FPC-05F-6PH20, symbol CORE:FPC-05F-6PH20
Connections:
- net +3.3V: now also FPC1.2
- net CTP_INT: now also FPC1.4
- net CTP_RST: now also FPC1.1
- net CTP_SCL: now also FPC1.6
- net CTP_SDA: now also FPC1.5
- net GND: now also FPC1.3, FPC1.7, FPC1.8
Changed lines of the file:
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@@
-	(wire
-		(pts
-			(xy 135.89 125.73) (xy 137.16 125.73)
-		)
-		(stroke
-			(width 0)
-			(type default)
-		)
-	)
 	(wire
 		(pts
 			(xy 60.96 72.39) (xy 60.96 74.93)
-		)
-		(stroke
-			(width 0)
-			(type default)
-		)
-	)
-	(wire
-		(pts
-			(xy 135.89 138.43) (xy 137.16 138.43)
 		)
 		(stroke
@@
 	)
 	(symbol
+		(lib_id "CORE:FPC-05F-6PH20")
+		(at 129.54 132.08 0)
+		(unit 1)
+		(body_style 1)
+		(exclude_from_sim no)
+		(in_bom yes)
+		(on_board yes)
+		(in_pos_files yes)
+		(dnp no)
+		(fields_autoplaced yes)
+		(property "Reference" "FPC1"
+			(at 135.89 130.8099 0)
+			(show_name no)
+			(do_not_autoplace no)
+			(effects
+				(font
+					(size 1.27 1.27)
+				)
+				(justify left)
+			)
+		)
+		(property "Value" "FPC-05F-6PH20"
+			(at 135.89 133.3499 0)
+			(show_name no)
+			(do_not_autoplace no)
+			(effects
+				(font
+					(size 1.27 1.27)
+				)
+				(justify left)
+			)
+		)
+		(property "Footprint" "CORE:FPC-05F-6PH20"
+			(at 129.54 132.08 0)
+			(hide yes)
+			(show_name no)
+			(do_not_autoplace no)
+			(effects
+				(font
+					(size 1.27 1.27)
+				)
+			)
+		)
+		(property "Datasheet" "https://wmsc.lcsc.com/wmsc/upload/file/pdf/v2/lcsc/2109221030_XUNPU-FPC-05F-6PH20_C2856796.pdf"
+			(at 129.54 132.08 0)
+			(hide yes)
+			(show_name no)
+			(do_not_autoplace no)
+			(effects
+				(font
+					(size 1.27 1.27)
+				)
+			)
+		)
+		(property "Description" "-25℃~+85℃ 0.3mm 0.5mm 2mm 500mA 50V 6P Bottom Contact Hinged Lid Phosphor bronze Surface Mount, Right Angle Tin SMD,P=0.5mm,卧贴 FFC, FPC (Flat Flexible) Connector Assemblies ROHS"
+			(at 129.54 132.08 0)
+			(hide yes)
+			(show_name no)
+			(do_not_autoplace no)
+			(effects
+				(font
+					(size 1.27 1.27)
+				)
+			)
+		)
+		(property "LCSC" "C2856796"
+			(at 129.54 132.08 0)
+			(hide yes)
+			(show_name no)
+			(do_not_autoplace no)
+			(effects
+				(font
+					(size 1.27 1.27)
+				)
+			)
+		)
+		(property "Manufacturer" "XUNPU"
+			(at 129.54 132.08 0)
+			(hide yes)
+			(show_name no)
+			(do_not_autoplace no)
+			(effects
+				(font
+					(size 1.27 1.27)
+				)
+			)
+		)
+		(property "Manufacturer Part" "FPC-05F-6PH20"
+			(at 129.54 132.08 0)
+			(hide yes)
+			(show_name no)
+			(do_not_autoplace no)
+			(effects
+				(font
+					(size 1.27 1.27)
+				)
+			)
+		)
+		(pin "3"
+		)
+		(pin "5"
+		)
+		(pin "4"
+		)
+		(pin "8"
+		)
+		(pin "6"
+		)
+		(pin "1"
+		)
+		(pin "7"
+		)
+		(pin "2"
+		)
+		(instances
+			(project "CORE_Rev1.0"
+				(path "/c7438a17-8217-4925-98df-f8ca6801320f/f61d5a97-b8cb-48b7-b2d8-b1ec9597c5e7"
+					(reference "FPC1")
+					(unit 1)
+				)
+			)
+		)
+	)
+	(symbol
 		(lib_id "power:GND")
 		(at 118.11 57.15 270)
@@
 	(symbol
 		(lib_id "power:GND")
-		(at 137.16 138.43 90)
-		(mirror x)
+		(at 133.35 143.51 0)
+		(mirror y)
 		(unit 1)
 		(body_style 1)
@@
 		(fields_autoplaced yes)
 		(property "Reference" "#PWR091"
-			(at 143.51 138.43 0)
+			(at 133.35 149.86 0)
 			(hide yes)
 			(show_name no)
@@
 		)
 		(property "Value" "GND"
-			(at 142.24 138.43 0)
+			(at 133.35 148.59 0)
 			(hide yes)
 			(show_name no)
@@
 		)
 		(property "Footprint" ""
-			(at 137.16 138.43 0)
+			(at 133.35 143.51 0)
 			(hide yes)
 			(show_name no)
@@
 		)
 		(property "Datasheet" ""
-			(at 137.16 138.43 0)
+			(at 133.35 143.51 0)
 			(hide yes)
 			(show_name no)
@@
 		)
 		(property "Description" "Power symbol creates a global label with name \"GND\" , ground"
-			(at 137.16 138.43 0)
+			(at 133.35 143.51 0)
 			(hide yes)
 			(show_name no)
@@
 	(symbol
 		(lib_id "power:GND")
-		(at 137.16 125.73 90)
+		(at 133.35 120.65 0)
 		(mirror x)
 		(unit 1)
@@
 		(fields_autoplaced yes)
 		(property "Reference" "#PWR090"
-			(at 143.51 125.73 0)
+			(at 133.35 114.3 0)
 			(hide yes)
 			(show_name no)
@@
 		)
 		(property "Value" "GND"
-			(at 142.24 125.73 0)
+			(at 133.35 115.57 0)
 			(hide yes)
 			(show_name no)
@@
 		)
 		(property "Footprint" ""
-			(at 137.16 125.73 0)
+			(at 133.35 120.65 0)
 			(hide yes)
 			(show_name no)
@@
 		)
 		(property "Datasheet" ""
-			(at 137.16 125.73 0)
+			(at 133.35 120.65 0)
 			(hide yes)
 			(show_name no)
@@
 		)
 		(property "Description" "Power symbol creates a global label with name \"GND\" , ground"
-			(at 137.16 125.73 0)
+			(at 133.35 120.65 0)
 			(hide yes)
 			(show_name no)
@@
 					(unit 1)
 				)
-			)
-		)
-	)
-	(symbol
-		(lib_id "CORE:FPC-6P")
-		(at 127 121.92 0)
-		(unit 1)
-		(body_style 1)
-		(exclude_from_sim no)
-		(in_bom yes)
-		(on_board yes)
-		(in_pos_files yes)
-		(dnp no)
-		(fields_autoplaced yes)
-		(property "Reference" "U7"
-			(at 130.175 116.84 0)
-			(show_name no)
-			(do_not_autoplace no)
-			(effects
-				(font
-					(size 1.27 1.27)
-				)
-			)
-		)
-		(property "Value" "FPC-6P"
-			(at 130.175 119.38 0)
-			(show_name no)
-			(do_not_autoplace no)
-			(effects
-				(font
-					(size 1.27 1.27)
-				)
-			)
-		)
-		(property "Footprint" "CORE:FPC-05F-6PH20"
-			(at 127 121.92 0)
-			(hide yes)
-			(show_name no)
-			(do_not_autoplace no)
-			(effects
-				(font
-					(size 1.27 1.27)
-				)
-			)
-		)
-		(property "Datasheet" "https://wmsc.lcsc.com/wmsc/upload/file/pdf/v2/lcsc/2109221030_XUNPU-FPC-05F-6PH20_C2856796.pdf"
-			(at 127 121.92 0)
-			(hide yes)
-			(show_name no)
-			(do_not_autoplace no)
-			(effects
-				(font
-					(size 1.27 1.27)
-				)
-			)
-		)
-		(property "Description" ""
-			(at 127 121.92 0)
-			(hide yes)
-			(show_name no)
-			(do_not_autoplace no)
-			(effects
-				(font
-					(size 1.27 1.27)
-				)
-			)
-		)
-		(pin "5"
-		)
-		(pin "7"
-		)
-		(pin "3"
-		)
-		(pin "2"
-		)
-		(pin "4"
-		)
-		(pin "1"
-		)
-		(pin "6"
-		)
-		(pin "8"
-		)
-		(instances
-			(project "CORE_Rev1.0"
-				(path "/c7438a17-8217-4925-98df-f8ca6801320f/f61d5a97-b8cb-48b7-b2d8-b1ec9597c5e7"
-					(reference "U7")
-					(unit 1)
-				)

Commit message: sch update
Parts:
- C14: footprint Capacitor_SMD:C_0402_1005Metric -> CORE:C_0402_1005Metric; symbol Device:C -> CORE:C
- R24, R25, R26: footprint Resistor_SMD:R_0402_1005Metric -> CORE:R_0402_1005Metric; symbol Device:R -> CORE:R
Changed lines of the file:
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@@
 	)
 	(symbol
-		(lib_id "Device:C")
+		(lib_id "CORE:C")
 		(at 115.57 44.45 0)
 		(unit 1)
@@
 			)
 		)
-		(property "Footprint" "Capacitor_SMD:C_0402_1005Metric"
+		(property "Footprint" "CORE:C_0402_1005Metric"
 			(at 116.5352 48.26 0)
 			(hide yes)
@@
 	)
 	(symbol
-		(lib_id "Device:R")
+		(lib_id "CORE:R")
 		(at 69.85 58.42 90)
 		(unit 1)
@@
 			)
 		)
-		(property "Footprint" "Resistor_SMD:R_0402_1005Metric"
+		(property "Footprint" "CORE:R_0402_1005Metric"
 			(at 69.85 60.198 90)
 			(hide yes)
@@
 	)
 	(symbol
-		(lib_id "Device:R")
+		(lib_id "CORE:R")
 		(at 40.64 67.31 90)
 		(unit 1)
@@
 			)
 		)
-		(property "Footprint" "Resistor_SMD:R_0402_1005Metric"
+		(property "Footprint" "CORE:R_0402_1005Metric"
 			(at 40.64 69.088 90)
 			(hide yes)
@@
 	)
 	(symbol
-		(lib_id "Device:R")
+		(lib_id "CORE:R")
 		(at 52.07 74.93 90)
 		(unit 1)
@@
 			)
 		)
-		(property "Footprint" "Resistor_SMD:R_0402_1005Metric"
+		(property "Footprint" "CORE:R_0402_1005Metric"
 			(at 52.07 76.708 90)
 			(hide yes)
