File: hardware/schematic/v1.0/CORE_Rev1.0/Signal.kicad_sch (KiCad schematic)
At the start: 25 parts, among them J26 Conn_01x04_Socket, U10 IPEX1, U11 IPEX1, U13 IPEX1, U14 IPEX1, U15 IPEX1, U16 IPEX1, U17 IPEX1, U18 IPEX1, U19 IPEX1, U20 IPEX1, U21 IPEX1, U22 IPEX1, U23 IPEX1, U24 IPEX1, U25 IPEX1, U26 IPEX1, U27 IPEX1, U28 IPEX1, U4 IPEX1, U8 IPEX1, U9 IPEX1

Commit message: sch update
Parts:
- removed U10, U11, U13, U14, U15, U16, U17, U18, U19, U20, U21, U22, U23, U24, U25, U26, U27, U28, U4, U8, U9: IPEX1, Counter:JLC_IPEX-1, symbol Counter:IPEX1
- added U10, U11, U12, U13, U14, U15, U16, U17, U18, U19, U20, U21, U22, U23, U24, U25, U26, U4, U7, U8, U9: IPEX1, CORE:KH-IPEX-K501-29, symbol CORE:IPEX1
Connections:
- net CLK1_FS_N: now also U23.4 (SIG)
- net CLK1_FS_P: now also U22.4 (SIG)
- net CLK1_FX_N: now also U7.4 (SIG)
- net CLK1_FX_P: now also U4.4 (SIG)
- net CLK2_FS_N: now also U25.4 (SIG)
- net CLK2_FS_P: now also U24.4 (SIG)
- net CLK2_FX_N: now also U9.4 (SIG)
- net CLK2_FX_P: now also U8.4 (SIG)
- net CLK3_FX_N: now also U11.4 (SIG)
- net CLK3_FX_P: now also U10.4 (SIG)
- net CLK4_FX_N: now also U13.4 (SIG)
- net CLK4_FX_P: now also U12.4 (SIG)
- net CLK5_FX_N: now also U15.4 (SIG)
- net CLK5_FX_P: now also U14.4 (SIG)
- net CLK6_FX_N: now also U17.4 (SIG)
- net CLK6_FX_P: now also U16.4 (SIG)
- net CLK7_FX_N: now also U19.4 (SIG)
- net CLK7_FX_P: now also U18.4 (SIG)
- net CLK_10M: now also U26.4 (SIG)
- net CLK_FX8_N: now also U21.4 (SIG)
- net CLK_FX8_P: now also U20.4 (SIG)
- net GND: now also U10.1 (GND), U10.2 (GND), U10.3 (GND), U11.1 (GND), U11.2 (GND), U11.3 (GND), U12.1 (GND), U12.2 (GND), U12.3 (GND), U13.1 (GND), U13.2 (GND), U13.3 (GND), U14.1 (GND), U14.2 (GND), U14.3 (GND), U15.1 (GND), U15.2 (GND), U15.3 (GND), U16.1 (GND), U16.2 (GND), U16.3 (GND), U17.1 (GND), U17.2 (GND), U17.3 (GND), U18.1 (GND), U18.2 (GND), U18.3 (GND), U19.1 (GND), U19.2 (GND), U19.3 (GND), U20.1 (GND), U20.2 (GND), U20.3 (GND), U21.1 (GND), U21.2 (GND), U21.3 (GND), U22.1 (GND), U22.2 (GND), U22.3 (GND), U23.1 (GND), U23.2 (GND), U23.3 (GND), U24.1 (GND), U24.2 (GND), U24.3 (GND), U25.1 (GND), U25.2 (GND), U25.3 (GND), U26.1 (GND), U26.2 (GND), U26.3 (GND), U4.1 (GND), U4.2 (GND), U4.3 (GND), U7.1 (GND), U7.2 (GND), U7.3 (GND), U8.1 (GND), U8.2 (GND), U8.3 (GND), U9.1 (GND), U9.2 (GND), U9.3 (GND)

Commit message: sch update
Parts:
- C13: footprint Capacitor_SMD:C_0402_1005Metric -> CORE:C_0402_1005Metric; symbol Device:C -> CORE:C
- R41, R42: footprint Resistor_SMD:R_0402_1005Metric -> CORE:R_0402_1005Metric; symbol Device:R -> CORE:R
Changed lines of the file:
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@@
 	)
 	(symbol
-		(lib_id "Device:R")
+		(lib_id "CORE:R")
 		(at 243.84 153.67 90)
 		(unit 1)
@@
 			)
 		)
-		(property "Footprint" "Resistor_SMD:R_0402_1005Metric"
+		(property "Footprint" "CORE:R_0402_1005Metric"
 			(at 243.84 155.448 90)
 			(hide yes)
@@
 	)
 	(symbol
-		(lib_id "Device:R")
+		(lib_id "CORE:R")
 		(at 243.84 143.51 270)
 		(unit 1)
@@
 			)
 		)
-		(property "Footprint" "Resistor_SMD:R_0402_1005Metric"
+		(property "Footprint" "CORE:R_0402_1005Metric"
 			(at 243.84 141.732 90)
 			(hide yes)
@@
 	)
 	(symbol
-		(lib_id "Device:C")
+		(lib_id "CORE:C")
 		(at 250.19 148.59 0)
 		(unit 1)
@@
 			)
 		)
-		(property "Footprint" "Capacitor_SMD:C_0402_1005Metric"
+		(property "Footprint" "CORE:C_0402_1005Metric"
 			(at 251.1552 152.4 0)
 			(hide yes)
