File: hardware/schematic/v1.0/CORE_Rev1.0/Storage.kicad_sch (KiCad schematic)
At the start: 43 parts, among them J12 USB_C_Receptacle_USB2.0_16P, U1 TXS02612RTWR, U12 FT2232HL, U3 SD_Card, U6 93LC56BT-I_OT, X1 X322512MSB4SI

Commit message: sch update
Parts:
- removed U1: TXS02612RTWR, Counter:QFN24_RTW, symbol Counter:TXS02612RTWR
- removed U3: SD_Card, Counter:SIM-SMD_LX_XDFP-0090-012, symbol Counter:SD_Card
- added Card1: TF_PUSH, CORE:TF_PUSH, symbol CORE:TF_PUSH
- added U1: TXS02612RTWR, CORE:TXS02612RTWR, symbol CORE:TXS02612RTWR_1
Connections:
- net +1.8V: now also U1.5 (VCCA)
- net +3.3V: now also Card1.4 (VDD), U1.17 (VCCB1), U1.21 (VCCB0)
- net GND: now also Card1.10, Card1.11, Card1.12, Card1.13, Card1.6 (VSS), U1.11 (GND2), U1.2 (GND1), U1.25 (EPAD)
- net SD_CLK: now also U1.9 (CLKA)
- net SD_CMD: now also U1.4 (CMDA)
- net SD_D0: now also U1.6 (DAT0A)
- net SD_D1: now also U1.7 (DAT1A)
- net SD_D2: now also U1.1 (DAT2A)
- net SD_D3: now also U1.3 (DAT3A)
- net at R19.2: now also Card1.8 (DAT1), U1.16 (DAT1B0)
- net at R23.2: now also Card1.1 (DAT2), U1.23 (DAT2B0)
- net at R22.2: now also Card1.2 (CD/DAT3), U1.22 (DAT3B0)
- net at R21.2: now also Card1.3 (CMD), U1.20 (CMDB0)
- net at R20.2: now also Card1.7 (DAT0), U1.18 (DAT0B0)
- net at R16.2: now also Card1.CD
- net at R15.1: now also U1.24 (SEL)
- new net: Card1.5 (CLX), U1.19 (CLKB0)

Commit message: sch update
Parts:
- removed BOOT_CFG1: CSW-2P, Counter:CSW DIP-2P, symbol Counter:CSW-2P
- removed U12: FT2232HL, JLCImport:FT2232HL, symbol JLCImport:FT2232HL
- added BOOT_CFG1: CSW-2P, CORE:DSWB02LHGET, symbol CORE:CSW-2P
- added U3: FT2232HL, CORE:FT2232HL, symbol CORE:FT2232HL
Connections:
- net +3.3V: now also U3.12 (VCORE), U3.20 (VCCIO), U3.31 (VCCIO), U3.37 (VCORE), U3.4 (VPHY), U3.42 (VCCIO), U3.50 (VREGIN), U3.56 (VCCIO), U3.64 (VCORE), U3.9 (VPLL)
- net GND: now also BOOT_CFG1.1, BOOT_CFG1.2, U3.1 (GND), U3.10 (AGND), U3.11 (GND), U3.13 (TEST), U3.15 (GND), U3.25 (GND), U3.35 (GND), U3.47 (GND), U3.5 (GND), U3.51 (GND)
- net at R28.2: now also U3.8 (DP)
- net at R11.1, R13.1: now also BOOT_CFG1.3
- net at R32.1: now also U3.19 (ADBUS3)
- net at C25.2, X1.3: now also U3.3 (OSCO)
- net at R31.1: now also U3.18 (ADBUS2)
- net at R12.1, R14.1: now also BOOT_CFG1.4
- net at R29.1: now also U3.16 (ADBUS0)
- net at R30.1: now also U3.17 (ADBUS1)
- net at C24.2, X1.1: now also U3.2 (OSCI)
- net at R43.1: now also U3.38 (BDBUS0)
- net at R44.2: now also U3.39 (BDBUS1)
- net at R35.2: now also U3.6 (REF)
- net at R33.1, U6.3 (DI): now also U3.61 (EEDATA)
- net at U6.4 (CLK): now also U3.62 (EECLK)
- net at U6.5 (CS): now also U3.63 (EECS)
- net at R27.2: now also U3.7 (DM)

Commit message: sch update
Parts:
- removed J12: USB_C_Receptacle_USB2.0_16P, Connector_USB:USB_C_Receptacle_Palconn_UTC16-G, symbol Connector:USB_C_Receptacle_USB2.0_16P
- removed R38, R39: 5.1K, Resistor_SMD:R_0402_1005Metric, symbol Device:R
- added R46, R47: 5.1K, Resistor_SMD:R_0402_1005Metric, symbol Device:R
- added USB1: TYPE-C_16PIN_2MD_073, CORE:TYPE-C_16PIN_2MD_073, symbol CORE:TYPE-C_16PIN_2MD_073
Connections:
- net +VBUS: now also USB1.A4B9 (VBUS), USB1.B4A9 (VBUS)
- net GND: now also R46.2, R47.2, USB1.13 (EH), USB1.14 (EH), USB1.A1B12 (GND), USB1.B1A12 (GND)
- net at R28.1: now also USB1.A6 (Dp1), USB1.B6 (Dp2)
- net at R27.1: now also USB1.A7 (Dn1), USB1.B7 (Dn2)
- new net: R46.1, USB1.A5 (CC1)
- new net: R47.1, USB1.B5 (CC2)

Commit message: sch update
Parts:
- C2, C20, C23, C24, C25, C3, C4, C5: footprint Capacitor_SMD:C_0402_1005Metric -> CORE:C_0402_1005Metric; symbol Device:C -> CORE:C
- C21, C22: footprint Capacitor_SMD:C_0603_1608Metric -> CORE:C_0603_1608Metric; symbol Device:C -> CORE:C
- R11, R12, R13, R14, R15, R16, R17, R18, R19, R20, R21, R22, R23, R27, R28, R29, R30, R31, R32, R33, R34, R35, R43, R44, R46, R47: footprint Resistor_SMD:R_0402_1005Metric -> CORE:R_0402_1005Metric; symbol Device:R -> CORE:R
